File: Circuit-Kits/USB-Breakout-with-Reset/USB-Breakout-with-Reset.kicad_pcb (KiCad board)
At the start: 2 copper layers, 39.8 x 20.6 mm, 12 parts, among them J1 USB-MICRO, SW1 RESET

Commit message: Created PDF of release.
Parts:
- added C1: 1uf, Rewire_NonLego:CAP-DISC-D7.5MM-P5MM, F.Cu at (134.6, 103.7)
- moved R1 3.24 mm to (138.6, 111.0)
- moved R2 1.59 mm to (149.8, 105.8)
- moved R3 1.59 mm to (149.8, 108.8)
Routing:
- net VUSB: track 22.4 -> 28.8 mm
- net Net-(D1-Pad1): track 16.2 -> 19.4 mm
- net GND: track 1.78 -> 3.86 mm
- net Net-(D2-Pad1): track 14.1 -> 15.2 mm
Changed lines of the file:
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@@
 (kicad_pcb (version 4) (host pcbnew 4.0.4+e1-6308~48~ubuntu14.04.1-stable)
   (general
-    (links 16)
-    (no_connects 0)
-    (area 104.572999 74.854999 178.510001 123.265001)
+    (links 18)
+    (no_connects 2)
+    (area 126.123799 93.123799 166.076201 113.876201)
     (thickness 1.6)
     (drawings 47)
-    (tracks 37)
+    (tracks 49)
     (zones 0)
-    (modules 12)
+    (modules 13)
     (nets 8)
   )
@@
   )
   (setup
-    (last_trace_width 0.254)
+    (last_trace_width 0.3302)
     (user_trace_width 0.1524)
     (user_trace_width 0.254)
@@
   )
   (module Rewire_NonLego:RES-CARBONFILM-7MM (layer F.Cu)
-    (at 135.4 110.92 90)
+    (at 138.636 110.97 90)
     (descr "Resistor, Axial,  RM 7.62mm, 1/3W,")
     (tags "Resistor Axial RM 7.62mm 1/3W R3")
@@
   )
   (module Rewire_NonLego:RES-CARBONFILM-7MM (layer F.Cu)
-    (at 148.22 105.8 180)
+    (at 149.812 105.8 180)
     (descr "Resistor, Axial,  RM 7.62mm, 1/3W,")
     (tags "Resistor Axial RM 7.62mm 1/3W R3")
@@
   )
   (module Rewire_NonLego:RES-CARBONFILM-7MM (layer F.Cu)
-    (at 148.22 108.8 180)
+    (at 149.812 108.8 180)
     (descr "Resistor, Axial,  RM 7.62mm, 1/3W,")
     (tags "Resistor Axial RM 7.62mm 1/3W R3")
@@
       (net 3 "Net-(D2-Pad1)"))
   )
+  (module Rewire_NonLego:CAP-DISC-D7.5MM-P5MM (layer F.Cu)
+    (at 134.572 103.684 270)
+    (descr "Capacitor 7.5mm Disc, Pitch 5mm")
+    (tags Capacitor)
+    (fp_text reference C1 (at 2.45 0 270) (layer F.Fab)
+      (effects (font (size 1 1) (thickness 0.15)))
+    )
+    (fp_text value 1uf (at 2.5 3.5 270) (layer F.Fab) hide
+      (effects (font (size 1 1) (thickness 0.15)))
+    )
+    (fp_text user 1uF (at 2.714 0 270) (layer F.SilkS)
+      (effects (font (size 1 1) (thickness 0.15)))
+    )
+    (fp_line (start -1.5 -2.5) (end 6.5 -2.5) (layer F.Fab) (width 0.05))
+    (fp_line (start -1.5 2.5) (end -1.5 -2.5) (layer F.Fab) (width 0.05))
+    (fp_line (start 6.5 2.5) (end -1.5 2.5) (layer F.Fab) (width 0.05))
+    (fp_line (start 6.5 -2.5) (end 6.5 2.5) (layer F.Fab) (width 0.05))
+    (fp_line (start -1.5 -2.5) (end 6.5 -2.5) (layer F.CrtYd) (width 0.05))
+    (fp_line (start 6.5 -2.5) (end 6.5 2.5) (layer F.CrtYd) (width 0.05))
+    (fp_line (start 6.5 2.5) (end -1.5 2.5) (layer F.CrtYd) (width 0.05))
+    (fp_line (start -1.5 2.5) (end -1.5 -2.5) (layer F.CrtYd) (width 0.05))
+    (fp_line (start -1.25 -2.25) (end 6.25 -2.25) (layer F.SilkS) (width 0.15))
+    (fp_line (start 6.25 -2.25) (end 6.25 2.25) (layer F.SilkS) (width 0.15))
+    (fp_line (start 6.25 2.25) (end -1.25 2.25) (layer F.SilkS) (width 0.15))
+    (fp_line (start -1.25 2.25) (end -1.25 -2.25) (layer F.SilkS) (width 0.15))
+    (pad 1 thru_hole rect (at 0 0 270) (size 1.4 1.4) (drill 0.9) (layers *.Cu *.Mask F.SilkS)
+      (net 4 VUSB))
+    (pad 2 thru_hole circle (at 5 0 270) (size 1.4 1.4) (drill 0.9) (layers *.Cu *.Mask F.SilkS)
+      (net 1 GND))
+  )
   (gr_text "Rewire Circuit Kit\n11/20/16" (at 165.8 116.2) (layer F.Fab)
     (effects (font (size 1.016 1.016) (thickness 0.1524)) (justify right))
@@
   (gr_line (start 162 93.2) (end 130 93.2) (layer Edge.Cuts) (width 0.1524))
   (gr_arc (start 162 97.2) (end 162 93.2) (angle 90) (layer Edge.Cuts) (width 0.1524))
-  (gr_text 1.5K (at 135.4 107 90) (layer F.SilkS)
+  (gr_text 1.5K (at 138.636 107 90) (layer F.SilkS)
     (effects (font (size 1.016 1.016) (thickness 0.1524)))
   )
@@
     (effects (font (size 1.016 1.016) (thickness 0.1524)))
   )
-  (gr_text 66.5 (at 144.4 109) (layer F.SilkS)
-    (effects (font (size 1.016 1.016) (thickness 0.1524)))
-  )
-  (gr_text 66.5 (at 144.4 105.8) (layer F.SilkS)
+  (gr_text 66.5 (at 145.748 108.684) (layer F.SilkS)
+    (effects (font (size 1.016 1.016) (thickness 0.1524)))
+  )
+  (gr_text 66.5 (at 145.748 105.8) (layer F.SilkS)
     (effects (font (size 1.016 1.016) (thickness 0.1524)))
   )
@@
   (gr_line (start 120.523 82.55) (end 120.523 93.98) (angle 90) (layer Dwgs.User) (width 0.15))
   (gr_line (start 104.648 82.55) (end 120.523 82.55) (angle 90) (layer Dwgs.User) (width 0.15))
+  (segment (start 134.572 108.684) (end 132.884 108.684) (width 0.3302) (layer B.Cu) (net 1))
+  (segment (start 132.884 108.684) (end 132.6 108.4) (width 0.3302) (layer B.Cu) (net 1))
   (segment (start 130.825 108.4) (end 132.6 108.4) (width 0.3302) (layer F.Cu) (net 1))
   (via (at 132.6 108.4) (size 0.6858) (drill 0.3302) (layers F.Cu B.Cu) (net 1))
-  (segment (start 141.8 102.59492) (end 141.8 104.6) (width 0.3302) (layer F.Cu) (net 2))
-  (segment (start 141.8 104.6) (end 140.6 105.8) (width 0.3302) (layer F.Cu) (net 2))
-  (segment (start 135.4 103.3) (end 135.4 105.8) (width 0.3302) (layer F.Cu) (net 2))
-  (segment (start 134.75 106.45) (end 135.4 105.8) (width 0.3302) (layer F.Cu) (net 2))
-  (segment (start 135.4 105.8) (end 140.6 105.8) (width 0.3302) (layer F.Cu) (net 2))
-  (segment (start 130.825 106.45) (end 134.75 106.45) (width 0.3302) (layer F.Cu) (net 2))
-  (segment (start 142 111.8) (end 142 110.2) (width 0.3302) (layer F.Cu) (net 3))
-  (segment (start 142 110.2) (end 140.6 108.8) (width 0.3302) (layer F.Cu) (net 3))
-  (segment (start 130.825 107.0991) (end 134.4991 107.0991) (width 0.3302) (layer F.Cu) (net 3))
-  (segment (start 134.4991 107.0991) (end 135.4 108) (width 0.3302) (layer F.Cu) (net 3))
-  (segment (start 135.4 108) (end 139.8 108) (width 0.3302) (layer F.Cu) (net 3))
-  (segment (start 139.8 108) (end 140.6 108.8) (width 0.3302) (layer F.Cu) (net 3))
+  (segment (start 139.635489 104.349489) (end 141.176 104.349489) (width 0.3302) (layer F.Cu) (net 2))
+  (segment (start 141.176 104.349489) (end 141.562511 104.349489) (width 0.3302) (layer F.Cu) (net 2))
+  (segment (start 141.8 104.6) (end 141.426511 104.6) (width 0.3302) (layer F.Cu) (net 2))
+  (segment (start 141.426511 104.6) (end 141.176 104.349489) (width 0.3302) (layer F.Cu) (net 2))
+  (segment (start 142.192 105.8) (end 142.192 104.992) (width 0.3302) (layer F.Cu) (net 2))
+  (segment (start 142.192 104.992) (end 141.8 104.6) (width 0.3302) (layer F.Cu) (net 2))
+  (segment (start 141.8 102.59492) (end 141.8 104.112) (width 0.3302) (layer F.Cu) (net 2))
+  (segment (start 138.636 103.35) (end 139.635489 104.349489) (width 0.3302) (layer F.Cu) (net 2))
+  (segment (start 141.8 104.112) (end 141.8 104.6) (width 0.3302) (layer F.Cu) (net 2))
+  (segment (start 141.562511 104.349489) (end 141.8 104.112) (width 0.3302) (layer F.Cu) (net 2))
+  (segment (start 140.128508 106.45) (end 130.825 106.45) (width 0.3302) (layer F.Cu) (net 2))
+  (segment (start 142.192 105.8) (end 140.778508 105.8) (width 0.3302) (layer F.Cu) (net 2))
+  (segment (start 140.778508 105.8) (end 140.128508 106.45) (width 0.3302) (layer F.Cu) (net 2))
+  (segment (start 142 111.8) (end 142 108.992) (width 0.3302) (layer F.Cu) (net 3))
+  (segment (start 142 108.992) (end 142.192 108.8) (width 0.3302) (layer F.Cu) (net 3))
+  (segment (start 130.825 107.0991) (end 140.4911 107.0991) (width 0.3302) (layer F.Cu) (net 3))
+  (segment (start 140.4911 107.0991) (end 142.192 108.8) (width 0.3302) (layer F.Cu) (net 3))
+  (segment (start 132.211269 105.68799) (end 132.56801 105.68799) (width 0.3302) (layer B.Cu) (net 4))
+  (segment (start 132.56801 105.68799) (end 134.572 103.684) (width 0.3302) (layer B.Cu) (net 4))
+  (segment (start 135.4 110.92) (end 134.434 109.954) (width 0.254) (layer B.Cu) (net 4))
+  (segment (start 134.434 109.954) (end 134.400511 109.920511) (width 0.254) (layer B.Cu) (net 4))
+  (segment (start 135.4 110.92) (end 135.45 110.97) (width 0.3302) (layer B.Cu) (net 4))
+  (segment (start 135.45 110.97) (end 138.636 110.97) (width 0.3302) (layer B.Cu) (net 4))
   (segment (start 130.2 106.8) (end 131.31201 105.68799) (width 0.254) (layer B.Cu) (net 4))
   (segment (start 131.31201 105.68799) (end 132.211269 105.68799) (width 0.254) (layer B.Cu) (net 4))
   (segment (start 130.2 109) (end 130.2 106.8) (width 0.254) (layer B.Cu) (net 4))
   (segment (start 131.120511 109.920511) (end 130.2 109) (width 0.254) (layer B.Cu) (net 4))
-  (segment (start 135.4 110.92) (end 134.400511 109.920511) (width 0.254) (layer B.Cu) (net 4))
   (segment (start 134.400511 109.920511) (end 131.120511 109.920511) (width 0.254) (layer B.Cu) (net 4))
   (segment (start 130 97) (end 132.999999 99.999999) (width 0.508) (layer F.Cu) (net 4))
