File: Circuit-Kits/USB-Breakout-with-Reset/USB-Breakout-with-Reset.sch (KiCad schematic (older format))
At the start: 12 parts, among them J1 USB-MICRO, SW1 RESET

Commit message: Created PDF of release.
Parts:
- added C1: 1uf, Rewire_NonLego:CAP-DISC-D7.5MM-P5MM, symbol CAP-CER-1UF-16V-X7R-RADIAL
Connections:
- net GND: now also C1.2
- net VUSB: now also C1.1
Changed lines of the file:
@@
 L GND #PWR03
 U 1 1 5833CE85
-P 2700 3650
-F 0 "#PWR03" H 2700 3400 50  0001 C CNN
-F 1 "GND" H 2700 3500 50  0000 C CNN
-F 2 "" H 2700 3650 50  0000 C CNN
-F 3 "" H 2700 3650 50  0000 C CNN
-	1    2700 3650
+P 2700 3850
+F 0 "#PWR03" H 2700 3600 50  0001 C CNN
+F 1 "GND" H 2700 3700 50  0000 C CNN
+F 2 "" H 2700 3850 50  0000 C CNN
+F 3 "" H 2700 3850 50  0000 C CNN
+	1    2700 3850
 	1    0    0    -1
 $EndComp
@@
 	2625 3600 2700 3600
 Wire Wire Line
-	2700 3600 2700 3650
-Wire Wire Line
-	2625 3200 2700 3200
+	2700 3600 2700 3850
+Wire Wire Line
+	2625 3200 2825 3200
 Wire Wire Line
 	2700 3200 2700 3100
@@
 	0    1    1    0
 $EndComp
+$Comp
+L CAP-CER-1UF-16V-X7R-RADIAL C1
+U 1 1 5833A09E
+P 2825 3550
+F 0 "C1" H 2925 3600 50  0000 L CNN
+F 1 "1uf" H 2925 3500 50  0000 L CNN
+F 2 "Rewire_NonLego:CAP-DISC-D7.5MM-P5MM" H 2825 3200 50  0001 C CIN
+F 3 "https://product.tdk.com/info/en/documents/catalog/leadmlcc_conventional_fk_en.pdf" H 2825 3550 5   0001 C CNN
+F 4 "C_Disc_D7.5_P5" H 2825 3200 50  0001 C CIN "Package"
+F 5 "TDK" H 2825 3200 50  0001 C CIN "MF_Name"
+F 6 "FK28X7R1C105K" H 2825 3200 50  0001 C CIN "MF_PN"
+F 7 "Digikey" H 2825 3200 50  0001 C CIN "S1_Name"
+F 8 "445-8614-ND" H 2825 3200 50  0001 C CIN "S1_PN"
+F 9 "CAP CER 1UF 16V X7R RADIAL" H 2825 3200 50  0001 C CIN "Description"
+F 10 "Not Verified" H 2825 3200 50  0001 C CIN "Verified"
+	1    2825 3550
+	1    0    0    -1
+$EndComp
+Wire Wire Line
+	2700 3750 2825 3750
+Wire Wire Line
+	2825 3750 2825 3650
+Connection ~ 2700 3750
+Wire Wire Line
+	2825 3200 2825 3450
+Connection ~ 2700 3200
 $EndSCHEMATC
