File: Development/Template/rewire/rewire.kicad_pcb (KiCad board)
At the start: 2 copper layers, 23.6 x 31.6 mm, 1 part

Commit message: Finished template.
Parts:
- removed BT1: Battery, Wickerlib:CR2032-4x3-NO-ROTATE
Other:
- board outline removed
Changed lines of the file:
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@@
     (tracks 0)
     (zones 0)
-    (modules 1)
-    (nets 3)
+    (modules 0)
+    (nets 1)
   )
   (page USLetter)
   (title_block
-    (title "Title")
-    (date "2016-12-06")
-    (rev "v1.0")
+    (title Title)
+    (date 2016-12-06)
+    (rev v1.0)
     (company "All Rights Reserved")
     (comment 1 help@browndoggadgets.com)
@@
   )
   (net 0 "")
-  (net 1 GND)
-  (net 2 VCC)
   (net_class Default "This is the default net class."
     (clearance 0.254)
@@
     (add_net VCC)
   )
-  (module Wickerlib:CR2032-4x3-NO-ROTATE (layer F.Cu)
-    (at 138.9 105.9)
-    (fp_text reference BT1 (at 4 -8 90) (layer F.Fab) hide
-      (effects (font (size 1 1) (thickness 0.15)))
-    )
-    (fp_text value Battery (at 15.4 -4) (layer F.SilkS)
-      (effects (font (size 1 1) (thickness 0.15)))
-    )
-    (fp_text user %R (at 8 -8) (layer F.Fab)
-      (effects (font (size 1 1) (thickness 0.15)))
-    )
-    (fp_line (start -3.8 -16) (end -3.8 8) (layer Edge.Cuts) (width 0.1))
-    (fp_line (start 19.8 -16) (end 19.8 8) (layer Edge.Cuts) (width 0.1))
-    (fp_line (start 0 -19.8) (end 16 -19.8) (layer Edge.Cuts) (width 0.1))
-    (fp_arc (start 0 -16) (end -3.8 -16) (angle 90) (layer Edge.Cuts) (width 0.1))
-    (fp_arc (start 16 -16) (end 16 -19.8) (angle 90) (layer Edge.Cuts) (width 0.1))
-    (fp_arc (start 16 8) (end 19.8 8) (angle 90) (layer Edge.Cuts) (width 0.1))
-    (fp_arc (start 0 8) (end 0 11.8) (angle 90) (layer Edge.Cuts) (width 0.1))
-    (fp_line (start 0 11.8) (end 16 11.8) (layer Edge.Cuts) (width 0.1))
-    (fp_line (start -3.8 -16) (end -3.8 8) (layer F.Fab) (width 0.05))
-    (fp_line (start 19.8 -16) (end 19.8 8) (layer F.Fab) (width 0.05))
-    (fp_line (start 0 -19.8) (end 16 -19.8) (layer F.Fab) (width 0.05))
-    (fp_arc (start 0 -16) (end -3.8 -16) (angle 90) (layer F.Fab) (width 0.05))
-    (fp_arc (start 16 -16) (end 16 -19.8) (angle 90) (layer F.Fab) (width 0.05))
-    (fp_arc (start 16 8) (end 19.8 8) (angle 90) (layer F.Fab) (width 0.05))
-    (fp_arc (start 0 8) (end 0 11.8) (angle 90) (layer F.Fab) (width 0.05))
-    (fp_line (start 0 11.8) (end 16 11.8) (layer F.Fab) (width 0.05))
-    (fp_line (start 0 0) (end 8 0) (layer B.SilkS) (width 8))
-    (fp_line (start 8 8) (end 8 -16) (layer F.SilkS) (width 8))
-    (fp_line (start 8 -16) (end 0 -16) (layer B.Mask) (width 5))
-    (fp_line (start 8 8) (end 8 -16) (layer B.Mask) (width 5))
-    (fp_line (start 0 0) (end 8 0) (layer B.Mask) (width 5))
-    (fp_line (start 8 -16) (end 8 8) (layer B.Cu) (width 5))
-    (fp_line (start 0 -16) (end 8 -16) (layer B.Cu) (width 5))
-    (fp_line (start 0 0) (end 8 0) (layer B.Cu) (width 5))
-    (fp_line (start 16 8) (end 16 -16) (layer B.Cu) (width 5))
-    (fp_line (start 16 -16) (end 16 8) (layer B.Mask) (width 5))
-    (fp_line (start 0 -16) (end 8 -16) (layer B.SilkS) (width 8))
-    (fp_line (start 0 0) (end 0 8) (layer F.SilkS) (width 8))
-    (fp_line (start 0.1 -16) (end 8.1 -16) (layer F.SilkS) (width 8))
-    (fp_line (start 0 8) (end 8 8) (layer F.SilkS) (width 8))
-    (fp_line (start 0 8) (end 8 8) (layer B.Cu) (width 5))
-    (fp_line (start 0 8) (end 8 8) (layer B.Mask) (width 5))
-    (fp_line (start 0 8) (end 8 8) (layer B.SilkS) (width 8))
-    (fp_line (start 0 0) (end 8 0) (layer F.SilkS) (width 8))
-    (fp_line (start 0 8) (end 0 0) (layer B.SilkS) (width 8))
-    (fp_line (start 8 8) (end 8 -16) (layer B.SilkS) (width 8))
-    (fp_line (start 0 8) (end 8 8) (layer B.Cu) (width 5))
-    (fp_line (start 0 8) (end 0 0) (layer B.Cu) (width 5))
-    (fp_line (start 0 8) (end 0 0) (layer B.Mask) (width 5))
-    (pad GND thru_hole circle (at 8 -8) (size 6 6) (drill 4.98) (layers *.Cu *.Mask)
-      (net 1 GND))
-    (pad + thru_hole circle (at 0 -8) (size 6 6) (drill 4.98) (layers *.Cu)
-      (net 2 VCC))
-    (pad + thru_hole circle (at 16 -8) (size 6 6) (drill 4.98) (layers *.Cu B.Mask)
-      (net 2 VCC))
-    (pad + smd rect (at 18.2 -8) (size 2.6 5.56) (layers F.Cu F.Paste F.Mask)
-      (net 2 VCC))
-    (pad GND smd rect (at 7.996 -7.746) (size 9 13.8) (layers F.Cu F.Paste F.Mask)
-      (net 1 GND))
-    (pad + smd rect (at -2.2 -8) (size 2.6 5.56) (layers F.Cu F.Paste F.Mask)
-      (net 2 VCC))
-    (pad GND thru_hole circle (at 0 -16) (size 6 6) (drill 4.98) (layers *.Cu *.Mask)
-      (net 1 GND))
-    (pad GND thru_hole circle (at 8 -16) (size 6 6) (drill 4.98) (layers *.Cu *.Mask)
-      (net 1 GND))
-    (pad + thru_hole circle (at 16 -16) (size 6 6) (drill 4.98) (layers *.Cu B.Mask)
-      (net 2 VCC))
-    (pad GND thru_hole circle (at 0 0) (size 6 6) (drill 4.98) (layers *.Cu *.Mask)
-      (net 1 GND))
-    (pad GND thru_hole circle (at 8 0) (size 6 6) (drill 4.98) (layers *.Cu *.Mask)
-      (net 1 GND))
-    (pad + thru_hole circle (at 16 0) (size 6 6) (drill 4.98) (layers *.Cu B.Mask)
-      (net 2 VCC))
-    (pad GND thru_hole circle (at 0 8) (size 6 6) (drill 4.98) (layers *.Cu *.Mask)
-      (net 1 GND))
-    (pad GND thru_hole circle (at 8 8) (size 6 6) (drill 4.98) (layers *.Cu *.Mask)
-      (net 1 GND))
-    (pad + thru_hole circle (at 16 8) (size 6 6) (drill 4.98) (layers *.Cu B.Mask)
-      (net 2 VCC))
-  )
   (gr_circle (center 117.348 76.962) (end 118.618 76.962) (layer Dwgs.User) (width 0.15))
