File: Circuit-Kits/Modules/2x3-LED-TH-Magnet/2x3-LED-TH-Magnet.sch (KiCad schematic (older format))
At the start: 1 part

Commit message: Converted modules to "Crazy Circuits".
Parts:
- LED1: footprint Rewire_Circuits:LED-10MMD-5MMP-TH-2x3 -> Crazy_Circuits:LED-10MMD-5MMP-TH-2x3
Changed lines of the file:
@@
 EESchema Schematic File Version 2
-LIBS:rewire_circuits
+LIBS:crazy_circuits
 LIBS:2x3-LED-TH-Magnet-cache
 EELAYER 25 0
@@
 F 0 "LED1" H 5050 3600 50  0000 L CNN
 F 1 "GREEN" H 5050 3500 50  0000 L CNN
-F 2 "Rewire_Circuits:LED-10MMD-5MMP-TH-2x3" H 4675 3425 50  0001 C CIN
+F 2 "Crazy_Circuits:LED-10MMD-5MMP-TH-2x3" H 4675 3425 50  0001 C CIN
 F 3 "" V 4675 3625 10  0001 C CNN
 F 4 "LED GREEN 10MM DIA 5MM PITCH TH" H 4675 3625 60  0001 C CNN "Description"
