File: Circuit-Kits/Modules/2x3-Potentiometer-P160K-TH/2x3-Potentiometer-P160K-TH.sch (KiCad schematic (older format))
At the start: 0 parts

Commit message: Added potentiometer 2x3
Parts:
- added R1: TRIMPOT-10K-3PIN-TH-0.20W-P160KN, Crazy_Circuits:POTENTIOMETER-P160K-2x3, symbol TRIMPOT-10K-3PIN-TH-0.20W-P160KN
Changed lines of the file:
@@
 EESchema Schematic File Version 2
-LIBS:rewire_circuits
+LIBS:crazy_circuits
+LIBS:wickerlib
+LIBS:2x3-Potentiometer-P160K-TH-cache
 EELAYER 25 0
 EELAYER END
@@
 Title "2x3 Potentiometer (P160K) Module"
 Date "18 Jan 2017"
-Rev"1.0"
-Comp "All rights reserved.")
-Comment1 "help@browndoggadgets.com")
-Comment2 "http://browndoggadgets.com/")
-Comment3 "Brown Dog Gadgets")
+Rev "1.0"
+Comp "All rights reserved."
+Comment1 "help@browndoggadgets.com"
+Comment2 "http://browndoggadgets.com/"
+Comment3 "Brown Dog Gadgets"
 Comment4 ""
 $EndDescr
+$Comp
+L TRIMPOT-10K-3PIN-TH-0.20W-P160KN R1
+U 1 1 588076C6
+P 5075 3150
+F 0 "R1" H 4975 3200 50  0000 R CNN
+F 1 "TRIMPOT-10K-3PIN-TH-0.20W-P160KN" H 4975 3100 50  0000 R CNN
+F 2 "Crazy_Circuits:POTENTIOMETER-P160K-2x3" H 5075 2800 50  0001 C CIN
+F 3 "http://www.bitechnologies.com/pdfs/p160.pdf" V 5075 3150 5   0001 C CNN
+F 4 "POT 10K OHM 1/5W PLASTIC LINEAR" H 5075 2800 50  0001 C CIN "Description"
+F 5 "TT Electronics" H 5075 2800 50  0001 C CIN "MF_Name"
+F 6 "P160KN-0QC15B10K" H 5075 2800 50  0001 C CIN "MF_PN"
+F 7 "Digikey" H 5075 2800 50  0001 C CIN "S1_Name"
+F 8 "987-1301-ND" H 5075 2800 50  0001 C CIN "S1_PN"
+	1    5075 3150
+	1    0    0    -1
+$EndComp
 $EndSCHEMATC
