File: Circuit-Kits/Modules/1x4-CR2032/1x4-CR2032.sch (KiCad schematic (older format))
At the start: 1 part

Commit message: Changed to BK-912 battery holder.
Parts:
- BT1: MF_Name Harwin -> MPD; MF_PN S8211-46R -> BK-912; S1_PN 952-1735-1-ND -> BK-912-ND
Changed lines of the file:
@@
 EESchema Schematic File Version 2
 LIBS:crazy_circuits
+LIBS:1x4-CR2032-cache
 EELAYER 25 0
 EELAYER END
@@
 F 3 "" V 4825 3740 50  0000 C CNN
 F 4 "HOLDER BATT COIN CR2032/20MM" H 4825 3700 60  0001 C CNN "Description"
-F 5 "Harwin" H 4825 3700 60  0001 C CNN "MF_Name"
-F 6 "S8211-46R" H 4825 3700 60  0001 C CNN "MF_PN"
+F 5 "MPD" H 4825 3700 60  0001 C CNN "MF_Name"
+F 6 "BK-912" H 4825 3700 60  0001 C CNN "MF_PN"
 F 7 "Digikey" H 4825 3700 60  0001 C CNN "S1_Name"
-F 8 "952-1735-1-ND" H 4825 3700 60  0001 C CNN "S1_PN"
+F 8 "BK-912-ND" H 4825 3700 60  0001 C CNN "S1_PN"
 	1    4825 3700
 	1    0    0    -1
