File: Circuit-Kits/Modules/1x2-Logo-Crazy-Circuits/1x2-Logo-Crazy-Circuits.kicad_pcb (KiCad board)
At the start: 2 copper layers, 15.6 x 7.8 mm, 1 part

Commit message: Public release of 1x2 Logo
Parts:
- moved LOGO 125.6 mm to (27.3, 43.2)
Other:
- board text added: "FABRICATION NOTES 1. THIS IS A 2 LAYER BOARD. 2. EXTERNAL LAYERS SHALL HAVE 1 OZ COPPER. 3. MATERIAL: FR4 AND 0.062 INCH +/- 10% THICK. 4. BOARDS SHALL BE ROHS COMPLIANT. 5. MANUFACTURE IN ACCORDANCE WITH IPC-6012 CLASS 2 6. MASK: BOTH SIDES OF THE BOARD SHALL HAVE SOLDER MASK (BLUE) OVER BARE COPPER. 7. SILK: BOTH SIDES OF THE BOARD SHALL HAVE WHITE SILK. DO NOT PLACE SILK OVER BARE COPPER. 8. F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"
Changed lines of the file:
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@@
     (area 104.572999 74.854999 178.510001 123.265001)
     (thickness 1.6)
-    (drawings 19)
+    (drawings 5)
     (tracks 0)
     (zones 0)
@@
   )
   (module Crazy_Circuits:LOGO-CRAZY-1x2 (layer F.Cu)
-    (at 141.097 96.393)
+    (at 27.305 43.18)
     (descr LOGO)
     (tags LOGO)
@@
     (pad BG smd oval (at 0 -3.937) (size 15.24 7.62) (layers F.Cu))
   )
-  (gr_text CIRCUITS (at 141.859 93.599) (layer F.Mask)
+  (dimension 7.8232 (width 0.1524) (layer Dwgs.User)
+    (gr_text "0.3080 in" (at 43.815 39.2938 270) (layer Dwgs.User)
+      (effects (font (size 1.016 1.016) (thickness 0.1524)))
+    )
+    (feature1 (pts (xy 29.6672 43.2054) (xy 44.6278 43.2054)))
+    (feature2 (pts (xy 29.6672 35.3822) (xy 44.6278 35.3822)))
+    (crossbar (pts (xy 43.0022 35.3822) (xy 43.0022 43.2054)))
+    (arrow1a (pts (xy 43.0022 43.2054) (xy 42.415779 42.078896)))
+    (arrow1b (pts (xy 43.0022 43.2054) (xy 43.588621 42.078896)))
+    (arrow2a (pts (xy 43.0022 35.3822) (xy 42.415779 36.508704)))
+    (arrow2b (pts (xy 43.0022 35.3822) (xy 43.588621 36.508704)))
+  )
+  (dimension 15.5956 (width 0.1524) (layer Dwgs.User)
+    (gr_text "0.6140 in" (at 27.305 31.877) (layer Dwgs.User)
+      (effects (font (size 1.016 1.016) (thickness 0.1524)))
+    )
+    (feature1 (pts (xy 35.1028 39.2684) (xy 35.1028 31.0642)))
+    (feature2 (pts (xy 19.5072 39.2684) (xy 19.5072 31.0642)))
+    (crossbar (pts (xy 19.5072 32.6898) (xy 35.1028 32.6898)))
+    (arrow1a (pts (xy 35.1028 32.6898) (xy 33.976296 33.276221)))
+    (arrow1b (pts (xy 35.1028 32.6898) (xy 33.976296 32.103379)))
+    (arrow2a (pts (xy 19.5072 32.6898) (xy 20.633704 33.276221)))
+    (arrow2b (pts (xy 19.5072 32.6898) (xy 20.633704 32.103379)))
+  )
+  (gr_text "FABRICATION NOTES\n\n1. THIS IS A 2 LAYER BOARD. \n2. EXTERNAL LAYERS SHALL HAVE 1 OZ COPPER.\n3. MATERIAL: FR4 AND 0.062 INCH +/- 10% THICK.\n4. BOARDS SHALL BE ROHS COMPLIANT. \n5. MANUFACTURE IN ACCORDANCE WITH IPC-6012 CLASS 2\n6. MASK: BOTH SIDES OF THE BOARD SHALL HAVE \n   SOLDER MASK (BLUE) OVER BARE COPPER. \n7. SILK: BOTH SIDES OF THE BOARD SHALL HAVE WHITE SILK. \n   DO NOT PLACE SILK OVER BARE COPPER.\n8. FINISH: ENIG.\n9. MINIMUM TRACE WIDTH - 0.006 INCH.\n   MINIMUM SPACE - 0.006 INCH.\n   MINIMUM HOLE DIA - 0.013 INCH. \n10. MAX HOLE PLACEMENT TOLERANCE OF +/- 0.003 INCH.\n11. MAX HOLE DIAMETER TOLERANCE OF +/- 0.003 INCH AFTER PLATING." (at 19.8882 87.6554) (layer Dwgs.User)
+    (effects (font (size 2.54 2.54) (thickness 0.254)) (justify left))
+  )
+  (gr_text CIRCUITS (at 28.067 40.386) (layer F.Mask)
     (effects (font (size 1.3 1.3) (thickness 0.3)))
   )
-  (gr_text CRAZY (at 139.319 91.313) (layer F.Mask)
+  (gr_text CRAZY (at 25.527 38.1) (layer F.Mask)
     (effects (font (size 1.3 1.3) (thickness 0.3)))
   )
-  (gr_circle (center 117.348 76.962) (end 118.618 76.962) (layer Dwgs.User) (width 0.15))
-  (gr_line (start 114.427 78.994) (end 114.427 74.93) (angle 90) (layer Dwgs.User) (width 0.15))
-  (gr_line (start 120.269 78.994) (end 114.427 78.994) (angle 90) (layer Dwgs.User) (width 0.15))
-  (gr_line (start 120.269 74.93) (end 120.269 78.994) (angle 90) (layer Dwgs.User) (width 0.15))
-  (gr_line (start 114.427 74.93) (end 120.269 74.93) (angle 90) (layer Dwgs.User) (width 0.15))
-  (gr_line (start 120.523 93.98) (end 104.648 93.98) (angle 90) (layer Dwgs.User) (width 0.15))
-  (gr_line (start 173.355 102.235) (end 173.355 94.615) (angle 90) (layer Dwgs.User) (width 0.15))
-  (gr_line (start 178.435 102.235) (end 173.355 102.235) (angle 90) (layer Dwgs.User) (width 0.15))
-  (gr_line (start 178.435 94.615) (end 178.435 102.235) (angle 90) (layer Dwgs.User) (width 0.15))
-  (gr_line (start 173.355 94.615) (end 178.435 94.615) (angle 90) (layer Dwgs.User) (width 0.15))
-  (gr_line (start 109.093 123.19) (end 109.093 114.3) (angle 90) (layer Dwgs.User) (width 0.15))
-  (gr_line (start 122.428 123.19) (end 109.093 123.19) (angle 90) (layer Dwgs.User) (width 0.15))
-  (gr_line (start 122.428 114.3) (end 122.428 123.19) (angle 90) (layer Dwgs.User) (width 0.15))
-  (gr_line (start 109.093 114.3) (end 122.428 114.3) (angle 90) (layer Dwgs.User) (width 0.15))
-  (gr_line (start 104.648 93.98) (end 104.648 82.55) (angle 90) (layer Dwgs.User) (width 0.15))
-  (gr_line (start 120.523 82.55) (end 120.523 93.98) (angle 90) (layer Dwgs.User) (width 0.15))
-  (gr_line (start 104.648 82.55) (end 120.523 82.55) (angle 90) (layer Dwgs.User) (width 0.15))
 )
