File: Circuit-Kits/Modules/2x3-USB-Power-Connector/2x3-USB-Power-Connector.sch (KiCad schematic (older format))
At the start: 4 parts, among them J1 MICRO-B, U1 MIC5365 3.3V

Commit message: Port project to KiCad 5.0
Parts:
- C1, C2: symbol CAP-CER-1UF-25V-X7R-0603 -> crazy_circuits:CAP-CER-1UF-25V-X7R-0603
- J1: symbol CONN-USB-MICRO-B-10118193 -> crazy_circuits:CONN-USB-MICRO-B-10118193
- U1: symbol IC-REG-LDO-3.3V-0.15A-MIC5365-SOT353 -> crazy_circuits:IC-REG-LDO-3.3V-0.15A-MIC5365-SOT353
Connections:
- wire segments 11 -> 16
Changed lines of the file:
@@
-EESchema Schematic File Version 2
+EESchema Schematic File Version 4
 LIBS:crazy_circuits
 LIBS:wickerlib
-EELAYER 25 0
+EELAYER 26 0
 EELAYER END
 $Descr USLetter 11000 8500
@@
 $EndDescr
 $Comp
-L GND #PWR01
+L crazy_circuits:GND #PWR01
 U 1 1 5833208F
 P 3050 4275
@@
 	2925 4225 3050 4225
 Wire Wire Line
-	3050 4125 3050 4275
+	3050 4125 3050 4225
 $Comp
-L CONN-USB-MICRO-B-10118193 J1
+L crazy_circuits:CONN-USB-MICRO-B-10118193 J1
 U 1 1 58844117
 P 2575 4025
@@
 $EndComp
 $Comp
-L GND #PWR02
+L crazy_circuits:GND #PWR02
 U 1 1 588A4DE7
 P 3750 4250
@@
 Connection ~ 3275 3825
 $Comp
-L CAP-CER-1UF-25V-X7R-0603 C1
+L crazy_circuits:CAP-CER-1UF-25V-X7R-0603 C1
 U 1 1 588A4E13
 P 3050 4025
@@
 Connection ~ 3050 4225
 $Comp
-L CAP-CER-1UF-25V-X7R-0603 C2
+L crazy_circuits:CAP-CER-1UF-25V-X7R-0603 C2
 U 1 1 588A4EC6
 P 4300 4025
@@
 $EndComp
 Wire Wire Line
-	4150 3825 4600 3825
+	4150 3825 4300 3825
 Wire Wire Line
 	4300 3925 4300 3825
 Connection ~ 4300 3825
 Wire Wire Line
-	3050 3725 3050 3925
+	3050 3725 3050 3825
 Connection ~ 3050 3825
 $Comp
-L GND #PWR03
+L crazy_circuits:GND #PWR03
 U 1 1 588A4F53
 P 4300 4250
@@
 	4600 3825 4600 3750
 $Comp
-L VCC #PWR04
+L crazy_circuits:VCC #PWR04
 U 1 1 588A5060
 P 4600 3750
@@
 $EndComp
 $Comp
-L IC-REG-LDO-3.3V-0.15A-MIC5365-SOT353 U1
+L crazy_circuits:IC-REG-LDO-3.3V-0.15A-MIC5365-SOT353 U1
 U 1 1 588A5298
 P 3750 3875
@@
 $EndComp
 $Comp
-L VIN #PWR05
+L crazy_circuits:VIN #PWR05
 U 1 1 588A55BE
 P 3050 3725
@@
 $EndComp
 Wire Wire Line
-	2925 3825 3350 3825
+	2925 3825 3050 3825
+Wire Wire Line
+	3275 3825 3350 3825
+Wire Wire Line
+	3050 4225 3050 4275
+Wire Wire Line
+	4300 3825 4600 3825
+Wire Wire Line
+	3050 3825 3050 3925
+Wire Wire Line
+	3050 3825 3275 3825
 $EndSCHEMATC
