File: Circuit-Kits/Modules/2x2-LED-RGB-TH-4PIN/2x2-LED-RGB-TH-4PIN.kicad_pcb (KiCad board)
At the start: 2 copper layers, 15.6 x 15.6 mm, 1 part

Commit message: Public release.
Parts:
- moved LED1 131.5 mm to (23.2, 44.4)
Other:
- board text added: "FABRICATION NOTES 1. THIS IS A 2 LAYER BOARD. 2. EXTERNAL LAYERS SHALL HAVE 1 OZ COPPER. 3. MATERIAL: FR4 AND 0.062 INCH +/- 10% THICK. 4. BOARDS SHALL BE ROHS COMPLIANT. 5. MANUFACTURE IN ACCORDANCE WITH IPC-6012 CLASS 2 6. MASK: BOTH SIDES OF THE BOARD SHALL HAVE SOLDER MASK (BLACK) OVER BARE COPPER. 7. SILK: BOTH SIDES OF THE BOARD SHALL HAVE WHITE SILK. DO NOT PLACE SILK OVER BARE COPPER. 8. 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"
Changed lines of the file:
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@@
     (area 104.572999 74.854999 178.510001 123.265001)
     (thickness 1.6)
-    (drawings 17)
+    (drawings 1)
     (tracks 0)
     (zones 0)
@@
   )
   (module Crazy_Circuits:LED-RGB-2.54MM-4PIN-2x2 (layer F.Cu)
-    (at 144.6276 94.67596)
+    (at 23.1658 44.3738)
     (descr "LED 5mm round vertical")
     (tags "LED 5mm round vertical")
@@
       (effects (font (size 1 1) (thickness 0.15)))
     )
-    (fp_line (start 4.064 -10.287) (end 0 -7.747) (layer F.Mask) (width 2))
+    (fp_line (start 4.064 -10.287) (end 0 -7.747) (layer F.SilkS) (width 2))
     (fp_arc (start 0.195441 -0.199792) (end 0 3.8) (angle 84.2) (layer Edge.Cuts) (width 0.05))
     (fp_line (start 11.8 -8) (end 11.8 0) (layer Edge.Cuts) (width 0.05))
@@
     (fp_arc (start 0.199792 -7.804559) (end -3.8 -8) (angle 84.2) (layer F.Fab) (width 0.05))
     (fp_arc (start 7.804559 -7.800208) (end 8 -11.8) (angle 84.2) (layer F.Fab) (width 0.05))
-    (fp_line (start 4.064 -5.08) (end 8.255 -8.001) (layer F.Mask) (width 2.286))
-    (fp_line (start 8.255 0.381) (end 4.064 -2.413) (layer F.Mask) (width 2.286))
-    (fp_line (start 3.937 2.286) (end 0 0) (layer F.Mask) (width 2.286))
+    (fp_line (start 4.064 -5.08) (end 8.255 -8.001) (layer F.SilkS) (width 2.286))
+    (fp_line (start 8.255 0.381) (end 4.064 -2.413) (layer F.SilkS) (width 2.286))
+    (fp_line (start 3.937 2.286) (end 0 0) (layer F.SilkS) (width 2.286))
     (fp_line (start 4.064 -10.287) (end 0 -7.747) (layer F.Cu) (width 2))
     (fp_line (start 4.064 -5.08) (end 8.255 -8.001) (layer F.Cu) (width 2.286))
@@
     (pad COM thru_hole rect (at 4 -5) (size 2 1.9) (drill 1.00076) (layers *.Cu *.Mask))
     (pad G thru_hole circle (at 4 -2.46 270) (size 1.9 1.9) (drill 1.00076) (layers *.Cu *.Mask))
-    (pad B thru_hole circle (at 0 0) (size 6 6) (drill 4.98) (layers *.Cu *.Mask))
-    (pad R thru_hole circle (at 0 -8) (size 6 6) (drill 4.98) (layers *.Cu *.Mask))
-    (pad COM thru_hole circle (at 8 -8) (size 6 6) (drill 4.98) (layers *.Cu *.Mask))
-    (pad G thru_hole circle (at 8 0) (size 6 6) (drill 4.98) (layers *.Cu *.Mask))
+    (pad B thru_hole circle (at 0 0) (size 6 6) (drill 4.98) (layers *.Cu B.Mask))
+    (pad R thru_hole circle (at 0 -8) (size 6 6) (drill 4.98) (layers *.Cu B.Mask))
+    (pad COM thru_hole circle (at 8 -8) (size 6 6) (drill 4.98) (layers *.Cu B.Mask))
+    (pad G thru_hole circle (at 8 0) (size 6 6) (drill 4.98) (layers *.Cu B.Mask))
     (pad B thru_hole circle (at 4 2.25 270) (size 1.9 1.9) (drill 1.00076) (layers *.Cu *.Mask))
     (pad R thru_hole circle (at 4 -10.25 270) (size 1.9 1.9) (drill 1.00076) (layers *.Cu *.Mask))
   )
-  (gr_circle (center 117.348 76.962) (end 118.618 76.962) (layer Dwgs.User) (width 0.15))
-  (gr_line (start 114.427 78.994) (end 114.427 74.93) (angle 90) (layer Dwgs.User) (width 0.15))
-  (gr_line (start 120.269 78.994) (end 114.427 78.994) (angle 90) (layer Dwgs.User) (width 0.15))
-  (gr_line (start 120.269 74.93) (end 120.269 78.994) (angle 90) (layer Dwgs.User) (width 0.15))
-  (gr_line (start 114.427 74.93) (end 120.269 74.93) (angle 90) (layer Dwgs.User) (width 0.15))
-  (gr_line (start 120.523 93.98) (end 104.648 93.98) (angle 90) (layer Dwgs.User) (width 0.15))
-  (gr_line (start 173.355 102.235) (end 173.355 94.615) (angle 90) (layer Dwgs.User) (width 0.15))
-  (gr_line (start 178.435 102.235) (end 173.355 102.235) (angle 90) (layer Dwgs.User) (width 0.15))
-  (gr_line (start 178.435 94.615) (end 178.435 102.235) (angle 90) (layer Dwgs.User) (width 0.15))
-  (gr_line (start 173.355 94.615) (end 178.435 94.615) (angle 90) (layer Dwgs.User) (width 0.15))
-  (gr_line (start 109.093 123.19) (end 109.093 114.3) (angle 90) (layer Dwgs.User) (width 0.15))
-  (gr_line (start 122.428 123.19) (end 109.093 123.19) (angle 90) (layer Dwgs.User) (width 0.15))
-  (gr_line (start 122.428 114.3) (end 122.428 123.19) (angle 90) (layer Dwgs.User) (width 0.15))
-  (gr_line (start 109.093 114.3) (end 122.428 114.3) (angle 90) (layer Dwgs.User) (width 0.15))
-  (gr_line (start 104.648 93.98) (end 104.648 82.55) (angle 90) (layer Dwgs.User) (width 0.15))
-  (gr_line (start 120.523 82.55) (end 120.523 93.98) (angle 90) (layer Dwgs.User) (width 0.15))
-  (gr_line (start 104.648 82.55) (end 120.523 82.55) (angle 90) (layer Dwgs.User) (width 0.15))
+  (gr_text "FABRICATION NOTES\n\n1. THIS IS A 2 LAYER BOARD. \n2. EXTERNAL LAYERS SHALL HAVE 1 OZ COPPER.\n3. MATERIAL: FR4 AND 0.062 INCH +/- 10% THICK.\n4. BOARDS SHALL BE ROHS COMPLIANT. \n5. MANUFACTURE IN ACCORDANCE WITH IPC-6012 CLASS 2\n6. MASK: BOTH SIDES OF THE BOARD SHALL HAVE \n   SOLDER MASK (BLACK) OVER BARE COPPER. \n7. SILK: BOTH SIDES OF THE BOARD SHALL HAVE WHITE SILK. \n   DO NOT PLACE SILK OVER BARE COPPER.\n8. FINISH: ENIG.\n9. MINIMUM TRACE WIDTH - 0.006 INCH.\n   MINIMUM SPACE - 0.006 INCH.\n   MINIMUM HOLE DIA - 0.013 INCH. \n10. MAX HOLE PLACEMENT TOLERANCE OF +/- 0.003 INCH.\n11. MAX HOLE DIAMETER TOLERANCE OF +/- 0.003 INCH AFTER PLATING." (at -2.0066 110.5408) (layer Dwgs.User)
+    (effects (font (size 2.54 2.54) (thickness 0.254)) (justify left))
+  )
 )
