File: Circuit-Kits/Modules/2x3-LED-RGB-SMT/2x3-LED-RGB-SMT.kicad_pcb (KiCad board)
At the start: 2 copper layers, 23.6 x 15.6 mm, 1 part

Commit message: Public release
Parts:
- moved LED1 126.2 mm to (24.8, 36.5)
Other:
- board text added: "FABRICATION NOTES 1. THIS IS A 2 LAYER BOARD. 2. EXTERNAL LAYERS SHALL HAVE 1 OZ COPPER. 3. MATERIAL: FR4 AND 0.062 INCH +/- 10% THICK. 4. BOARDS SHALL BE ROHS COMPLIANT. 5. MANUFACTURE IN ACCORDANCE WITH IPC-6012 CLASS 2 6. MASK: BOTH SIDES OF THE BOARD SHALL HAVE SOLDER MASK (BLACK) OVER BARE COPPER. 7. SILK: BOTH SIDES OF THE BOARD SHALL HAVE WHITE SILK. DO NOT PLACE SILK OVER BARE COPPER. 8. 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"
Changed lines of the file:
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@@
     (area 104.572999 74.854999 178.510001 123.265001)
     (thickness 1.6)
-    (drawings 17)
+    (drawings 1)
     (tracks 0)
     (zones 0)
@@
   )
   (module Crazy_Circuits:LED-RGB-0606-2x3 (layer F.Cu)
-    (at 131.574 103.79456)
+    (at 24.7924 36.5252)
     (descr "2.54mm pitch through hole centered 2x2")
     (fp_text reference LED1 (at 3.9 -2.3) (layer F.Fab)
@@
       (effects (font (size 1 1) (thickness 0.15)))
     )
-    (pad 3 thru_hole circle (at 0 0) (size 6 6) (drill 4.98) (layers *.Cu *.Mask)
-      (net 1 VCC))
-    (pad 1 thru_hole circle (at 0 -8) (size 6 6) (drill 4.98) (layers *.Cu *.Mask)
+    (pad 3 thru_hole circle (at 0 0) (size 6 6) (drill 4.98) (layers *.Cu B.Mask)
+      (net 1 VCC))
+    (pad 1 thru_hole circle (at 0 -8) (size 6 6) (drill 4.98) (layers *.Cu B.Mask)
       (net 2 /B))
-    (pad 3 thru_hole circle (at 8 0) (size 6 6) (drill 4.98) (layers *.Cu *.Mask)
+    (pad 3 thru_hole circle (at 8 0) (size 6 6) (drill 4.98) (layers *.Cu B.Mask)
       (net 1 VCC))
     (pad 3 smd rect (at 3 -3.6) (size 0.85 0.5) (layers F.Cu F.Paste F.Mask)
@@
     (pad 2 smd rect (at 4.75 -4.6) (size 0.85 0.5) (layers F.Cu F.Paste F.Mask)
       (net 4 /G))
-    (pad 2 thru_hole circle (at 8 -8) (size 6 6) (drill 4.98) (layers *.Cu *.Mask)
+    (pad 2 thru_hole circle (at 8 -8) (size 6 6) (drill 4.98) (layers *.Cu B.Mask)
       (net 4 /G))
-    (pad 4 thru_hole circle (at 16 -8) (size 6 6) (drill 4.98) (layers *.Cu *.Mask)
+    (pad 4 thru_hole circle (at 16 -8) (size 6 6) (drill 4.98) (layers *.Cu B.Mask)
       (net 3 /R))
-    (pad 3 thru_hole circle (at 16 0) (size 6 6) (drill 4.98) (layers *.Cu *.Mask)
-      (net 1 VCC))
-  )
-  (gr_circle (center 117.348 76.962) (end 118.618 76.962) (layer Dwgs.User) (width 0.15))
-  (gr_line (start 114.427 78.994) (end 114.427 74.93) (angle 90) (layer Dwgs.User) (width 0.15))
-  (gr_line (start 120.269 78.994) (end 114.427 78.994) (angle 90) (layer Dwgs.User) (width 0.15))
-  (gr_line (start 120.269 74.93) (end 120.269 78.994) (angle 90) (layer Dwgs.User) (width 0.15))
-  (gr_line (start 114.427 74.93) (end 120.269 74.93) (angle 90) (layer Dwgs.User) (width 0.15))
-  (gr_line (start 120.523 93.98) (end 104.648 93.98) (angle 90) (layer Dwgs.User) (width 0.15))
-  (gr_line (start 173.355 102.235) (end 173.355 94.615) (angle 90) (layer Dwgs.User) (width 0.15))
-  (gr_line (start 178.435 102.235) (end 173.355 102.235) (angle 90) (layer Dwgs.User) (width 0.15))
-  (gr_line (start 178.435 94.615) (end 178.435 102.235) (angle 90) (layer Dwgs.User) (width 0.15))
-  (gr_line (start 173.355 94.615) (end 178.435 94.615) (angle 90) (layer Dwgs.User) (width 0.15))
-  (gr_line (start 109.093 123.19) (end 109.093 114.3) (angle 90) (layer Dwgs.User) (width 0.15))
-  (gr_line (start 122.428 123.19) (end 109.093 123.19) (angle 90) (layer Dwgs.User) (width 0.15))
-  (gr_line (start 122.428 114.3) (end 122.428 123.19) (angle 90) (layer Dwgs.User) (width 0.15))
-  (gr_line (start 109.093 114.3) (end 122.428 114.3) (angle 90) (layer Dwgs.User) (width 0.15))
-  (gr_line (start 104.648 93.98) (end 104.648 82.55) (angle 90) (layer Dwgs.User) (width 0.15))
-  (gr_line (start 120.523 82.55) (end 120.523 93.98) (angle 90) (layer Dwgs.User) (width 0.15))
-  (gr_line (start 104.648 82.55) (end 120.523 82.55) (angle 90) (layer Dwgs.User) (width 0.15))
+    (pad 3 thru_hole circle (at 16 0) (size 6 6) (drill 4.98) (layers *.Cu B.Mask)
+      (net 1 VCC))
+  )
+  (gr_text "FABRICATION NOTES\n\n1. THIS IS A 2 LAYER BOARD. \n2. EXTERNAL LAYERS SHALL HAVE 1 OZ COPPER.\n3. MATERIAL: FR4 AND 0.062 INCH +/- 10% THICK.\n4. BOARDS SHALL BE ROHS COMPLIANT. \n5. MANUFACTURE IN ACCORDANCE WITH IPC-6012 CLASS 2\n6. MASK: BOTH SIDES OF THE BOARD SHALL HAVE \n   SOLDER MASK (BLACK) OVER BARE COPPER. \n7. SILK: BOTH SIDES OF THE BOARD SHALL HAVE WHITE SILK. \n   DO NOT PLACE SILK OVER BARE COPPER.\n8. FINISH: ENIG.\n9. MINIMUM TRACE WIDTH - 0.006 INCH.\n   MINIMUM SPACE - 0.006 INCH.\n   MINIMUM HOLE DIA - 0.013 INCH. \n10. MAX HOLE PLACEMENT TOLERANCE OF +/- 0.003 INCH.\n11. MAX HOLE DIAMETER TOLERANCE OF +/- 0.003 INCH AFTER PLATING." (at 1.3208 94.0308) (layer Dwgs.User)
+    (effects (font (size 2.54 2.54) (thickness 0.254)) (justify left))
+  )
 )
