File: Circuit-Kits/Modules/2x3-Speaker-TH-5mm-Pitch/2x3-Speaker-TH-5mm-Pitch.sch (KiCad schematic (older format))
At the start: 1 part

Commit message: Port project to KiCad 5.0
Parts:
- SPK1: symbol Speaker -> crazy_circuits:Speaker
Changed lines of the file:
@@
-EESchema Schematic File Version 2
-LIBS:2x3-Speaker-TH-5mm-Pitch-rescue
+EESchema Schematic File Version 4
 LIBS:crazy_circuits
-LIBS:2x3-Speaker-TH-5mm-Pitch-cache
-EELAYER 25 0
+EELAYER 26 0
 EELAYER END
 $Descr USLetter 11000 8500
@@
 $EndDescr
 $Comp
-L Speaker SPK1
+L crazy_circuits:Speaker SPK1
 U 1 1 58806521
 P 4825 3700
