File: Circuit-Kits/Modules/2x3-Slide-Switch-EG1218-TH/2x3-Slide-Switch-EG1218-TH.kicad_pcb (KiCad board)
At the start: 2 copper layers, 0 parts

Commit message: Release 2x3 Slide Switch EG1218 v1.0
Parts:
- added SW1: P/N EG1218, Crazy_Circuits:SWITCH-SPDT-3PIN-2.5mmPITCH-TH-2x3, F.Cu at (5.56, 41.2)
Other:
- board outline added: 23.5 x 15.6 mm
- board text added: "FABRICATION NOTES 1. THIS IS A 2 LAYER BOARD. 2. EXTERNAL LAYERS SHALL HAVE 1 OZ COPPER. 3. MATERIAL: FR4 AND 0.062 INCH +/- 10% THICK. 4. BOARDS SHALL BE ROHS COMPLIANT. 5. MANUFACTURE IN ACCORDANCE WITH IPC-6012 CLASS 2 6. MASK: BOTH SIDES OF THE BOARD SHALL HAVE SOLDER MASK (RED) OVER BARE COPPER. 7. SILK: BOTH SIDES OF THE BOARD SHALL HAVE WHITE SILKSCREEN. DO NOT PLACE SILK OVER BARE COPPER.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"
- board text removed: "FABRICATION NOTES 1. THIS IS A 2 LAYER BOARD. 2. EXTERNAL LAYERS SHALL HAVE 1 OZ COPPER. 3. MATERIAL: FR4 AND 0.062 INCH +/- 10% THICK. 4. BOARDS SHALL BE ROHS COMPLIANT. 5. MANUFACTURE IN ACCORDANCE WITH IPC-6012 CLASS 2 6. MASK: BOTH SIDES OF THE BOARD SHALL HAVE SOLDER MASK (ANY COLOR) OVER BARE COPPER. 7. SILK: BOTH SIDES OF THE BOARD SHALL HAVE WHITE SILKSCREEN. DO NOT PLACE SILK OVER BARE C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"
Changed lines of the file:
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@@
 (kicad_pcb (version 4) (host pcbnew 4.0.5-e0-6337~49~ubuntu16.04.1)
   (general
-    (links 0)
-    (no_connects 0)
-    (area 104.572999 74.854999 178.510001 123.265001)
+    (links 6)
+    (no_connects 6)
+    (area 1.361679 2.844323 144.734519 104.15524)
     (thickness 1.6)
     (drawings 1)
     (tracks 0)
     (zones 0)
-    (modules 0)
-    (nets 1)
+    (modules 1)
+    (nets 4)
   )
   (page USLetter)
@@
     (title "2x3 Slide Switch TH (EG1218)")
     (date "17 Mar 2017")
-    (rev "1.0")
+    (rev 1.0)
     (company "All rights reserved.")
-    (comment 1 "help@browndoggadgets.com")
-    (comment 2 "http://browndoggadgets.com/")
+    (comment 1 help@browndoggadgets.com)
+    (comment 2 http://browndoggadgets.com/)
     (comment 3 "Brown Dog Gadgets")
   )
@@
   )
   (net 0 "")
+  (net 1 /3)
+  (net 2 /1)
+  (net 3 /2)
   (net_class Default "This is the default net class."
     (clearance 0.254)
@@
     (uvia_dia 0.6858)
     (uvia_drill 0.3302)
+    (add_net /1)
+    (add_net /2)
+    (add_net /3)
   )
-  (gr_text "FABRICATION NOTES\n\n1. THIS IS A 2 LAYER BOARD. \n2. EXTERNAL LAYERS SHALL HAVE 1 OZ COPPER.\n3. MATERIAL: FR4 AND 0.062 INCH +/- 10% THICK.\n4. BOARDS SHALL BE ROHS COMPLIANT. \n5. MANUFACTURE IN ACCORDANCE WITH IPC-6012 CLASS 2\n6. MASK: BOTH SIDES OF THE BOARD SHALL HAVE \n   SOLDER MASK (ANY COLOR) OVER BARE COPPER. \n7. SILK: BOTH SIDES OF THE BOARD SHALL HAVE \n   WHITE SILKSCREEN. DO NOT PLACE SILK OVER BARE COPPER.\n8. FINISH: ENIG.\n9. MINIMUM TRACE WIDTH - 0.006 INCH.\n   MINIMUM SPACE - 0.006 INCH.\n   MINIMUM HOLE DIA - 0.013 INCH. \n10. MAX HOLE PLACEMENT TOLERANCE OF +/- 0.003 INCH.\n11. MAX HOLE DIAMETER TOLERANCE OF +/- 0.003 INCH AFTER PLATING." (at 120.3198 68.326) (layer Dwgs.User)
+  (module Crazy_Circuits:SWITCH-SPDT-3PIN-2.5mmPITCH-TH-2x3 (layer F.Cu)
+    (at 5.55952 41.21912)
+    (descr http://spec_sheets.e-switch.com/specs/P040040.pdf)
+    (tags "SWITCH SPDT EG1218 2x3")
+    (fp_text reference SW1 (at 7.9375 -3.8735) (layer F.Fab)
+      (effects (font (size 1 1) (thickness 0.15)))
+    )
+    (fp_text value "P/N EG1218" (at 8.2 4.8) (layer F.Fab) hide
+      (effects (font (size 1 1) (thickness 0.15)))
+    )
+    (fp_line (start 8.001 -7.5795) (end 8.001 -1.0795) (layer B.Mask) (width 1.5))
+    (fp_line (start 0 -8) (end 0 0) (layer B.Mask) (width 5))
+    (fp_text user "SLIDE " (at 4.0005 0 90) (layer F.SilkS)
+      (effects (font (size 1 1) (thickness 0.15)))
+    )
+    (fp_text user SWITCH (at 4 -8 90) (layer F.SilkS)
+      (effects (font (size 1 1) (thickness 0.15)))
+    )
+    (fp_line (start 7.9375 -8.1915) (end 7.9375 0) (layer F.SilkS) (width 1.5))
+    (fp_line (start 16 -8) (end 16 0) (layer B.Mask) (width 5))
+    (fp_line (start 0 -8) (end 0 0) (layer B.Cu) (width 5))
+    (fp_line (start 16 -8) (end 16 0) (layer B.Cu) (width 5))
+    (fp_line (start 8.001 -7.5795) (end 8.001 -1.0795) (layer B.Cu) (width 1.5))
+    (fp_arc (start 0.106632 -8.00018) (end -3.693368 -7.90018) (angle 89.9) (layer Edge.Cuts) (width 0.04064))
+    (fp_arc (start 0.111824 0) (end 0.411824 3.8) (angle 94.51398846) (layer Edge.Cuts) (width 0.04064))
+    (fp_arc (start 16 0) (end 19.8 -0.1) (angle 91.50743576) (layer Edge.Cuts) (width 0.04064))
+    (fp_arc (start 15.998684 -8) (end 15.898684 -11.8) (angle 91.50743576) (layer Edge.Cuts) (width 0.04064))
+    (fp_line (start 19.8 -8) (end 19.8 0) (layer Edge.Cuts) (width 0.04064))
+    (fp_line (start 16 -11.8) (end 0 -11.8) (layer Edge.Cuts) (width 0.04064))
+    (fp_line (start 16 3.8) (end 0.3 3.8) (layer Edge.Cuts) (width 0.04064))
+    (fp_line (start -3.7 -8) (end -3.7 0) (layer Edge.Cuts) (width 0.04064))
+    (fp_arc (start 0.106632 -8.00018) (end -3.693368 -7.90018) (angle 89.9) (layer F.Fab) (width 0.04064))
+    (fp_arc (start 0.111824 0) (end 0.411824 3.8) (angle 94.51398846) (layer F.Fab) (width 0.04064))
+    (fp_arc (start 16 0) (end 19.8 -0.1) (angle 91.50743576) (layer F.Fab) (width 0.04064))
+    (fp_arc (start 15.998684 -8) (end 15.898684 -11.8) (angle 91.50743576) (layer F.Fab) (width 0.04064))
+    (fp_line (start 19.8 -8) (end 19.8 0) (layer F.Fab) (width 0.04064))
+    (fp_line (start 16 -11.8) (end 0 -11.8) (layer F.Fab) (width 0.04064))
+    (fp_line (start 16 3.8) (end 0.3 3.8) (layer F.Fab) (width 0.04064))
+    (fp_line (start -3.7 -8) (end -3.7 0) (layer F.Fab) (width 0.04064))
+    (fp_line (start 0 -8.0645) (end 0 0) (layer F.SilkS) (width 2))
+    (fp_line (start 5.461 -4.0005) (end 0 -4.0005) (layer F.SilkS) (width 1.5))
+    (fp_line (start 15.9385 0.0635) (end 15.9385 -8.001) (layer F.SilkS) (width 2))
+    (fp_line (start 10.4775 -4.0005) (end 15.9385 -4.0005) (layer F.SilkS) (width 1.5))
+    (fp_line (start 5.461 -4.0005) (end 0 -4.0005) (layer B.Cu) (width 1.5))
+    (fp_line (start 5.461 -4.0005) (end 0 -4.0005) (layer B.Mask) (width 1.5))
+    (fp_line (start 15.9385 -4.0005) (end 10.4775 -4.0005) (layer B.Cu) (width 1.5))
+    (fp_line (start 15.9385 -4.0005) (end 10.4775 -4.0005) (layer B.Mask) (width 1.5))
+    (fp_line (start 7.9375 -6.604) (end 7.9375 -1.143) (layer B.Cu) (width 1.5))
+    (fp_line (start 7.9375 -6.604) (end 7.9375 -1.143) (layer B.Mask) (width 1.5))
+    (pad 3 thru_hole circle (at 16 -8) (size 6 6) (drill 4.98) (layers *.Cu B.Mask)
+      (net 1 /3))
+    (pad 1 thru_hole circle (at 0 0) (size 6 6) (drill 4.98) (layers *.Cu B.Mask)
+      (net 2 /1))
+    (pad 2 thru_hole circle (at 7.9394 -3.9751) (size 1.25 1.25) (drill 1) (layers *.Cu *.Mask)
+      (net 3 /2))
+    (pad 3 thru_hole circle (at 5.4394 -3.9751) (size 1.25 1.25) (drill 1) (layers *.Cu *.Mask)
+      (net 1 /3))
+    (pad 1 thru_hole circle (at 10.4394 -3.9751) (size 1.25 1.25) (drill 1) (layers *.Cu *.Mask)
+      (net 2 /1))
+    (pad 3 thru_hole circle (at 16 0) (size 6 6) (drill 4.98) (layers *.Cu B.Mask)
+      (net 1 /3))
+    (pad 1 thru_hole circle (at 0 -8) (size 6 6) (drill 4.98) (layers *.Cu B.Mask)
+      (net 2 /1))
+    (pad 2 thru_hole circle (at 8 -8) (size 6 6) (drill 4.98) (layers *.Cu B.Mask)
+      (net 3 /2))
+    (pad 2 thru_hole circle (at 8 0) (size 6 6) (drill 4.98) (layers *.Cu B.Mask)
+      (net 3 /2))
+  )
+  (gr_text "FABRICATION NOTES\n\n1. THIS IS A 2 LAYER BOARD. \n2. EXTERNAL LAYERS SHALL HAVE 1 OZ COPPER.\n3. MATERIAL: FR4 AND 0.062 INCH +/- 10% THICK.\n4. BOARDS SHALL BE ROHS COMPLIANT. \n5. MANUFACTURE IN ACCORDANCE WITH IPC-6012 CLASS 2\n6. MASK: BOTH SIDES OF THE BOARD SHALL HAVE \n   SOLDER MASK (RED) OVER BARE COPPER. \n7. SILK: BOTH SIDES OF THE BOARD SHALL HAVE \n   WHITE SILKSCREEN. DO NOT PLACE SILK OVER BARE COPPER.\n8. FINISH: ENIG.\n9. MINIMUM TRACE WIDTH - 0.006 INCH.\n   MINIMUM SPACE - 0.006 INCH.\n   MINIMUM HOLE DIA - 0.013 INCH. \n10. MAX HOLE PLACEMENT TOLERANCE OF +/- 0.003 INCH.\n11. MAX HOLE DIAMETER TOLERANCE OF +/- 0.003 INCH AFTER PLATING." (at 2.11328 95.7834) (layer Dwgs.User)
     (effects (font (size 2.54 2.54) (thickness 0.254)) (justify left))
   )
