File: Circuit-Kits/Modules/2x3-Push-Terminal-3mm-Pitch-SMT/2x3-Push-Terminal-3mm-Pitch-SMT.kicad_pcb (KiCad board)
At the start: 2 copper layers, 0 parts

Commit message: Releave v1.0 2x3, 2x2 Push Terminals.
Parts:
- added J1: Push Terminal Block, Crazy_Circuits:PUSH-TERMINAL-3MM-SMT-2x3, F.Cu at (3.96, 29.8)
Other:
- board outline added: 23.6 x 15.6 mm
- board text added: "FABRICATION NOTES 1. THIS IS A 2 LAYER BOARD. 2. EXTERNAL LAYERS SHALL HAVE 1 OZ COPPER. 3. MATERIAL: FR4 AND 0.062 INCH +/- 10% THICK. 4. BOARDS SHALL BE ROHS COMPLIANT. 5. MANUFACTURE IN ACCORDANCE WITH IPC-6012 CLASS 2 6. MASK: BOTH SIDES OF THE BOARD SHALL HAVE SOLDER MASK (PURPLE) OVER BARE COPPER. 7. SILK: BOTH SIDES OF THE BOARD SHALL HAVE WHITE SILKSCREEN. DO NOT PLACE SILK OVER BARE COPP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"
- board text removed: "FABRICATION NOTES 1. THIS IS A 2 LAYER BOARD. 2. EXTERNAL LAYERS SHALL HAVE 1 OZ COPPER. 3. MATERIAL: FR4 AND 0.062 INCH +/- 10% THICK. 4. BOARDS SHALL BE ROHS COMPLIANT. 5. MANUFACTURE IN ACCORDANCE WITH IPC-6012 CLASS 2 6. MASK: BOTH SIDES OF THE BOARD SHALL HAVE SOLDER MASK (ANY COLOR) OVER BARE COPPER. 7. SILK: BOTH SIDES OF THE BOARD SHALL HAVE WHITE SILKSCREEN. DO NOT PLACE SILK OVER BARE C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"
Changed lines of the file:
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@@
 (kicad_pcb (version 4) (host pcbnew 4.0.5-e0-6337~49~ubuntu16.04.1)
   (general
-    (links 0)
-    (no_connects 0)
-    (area 104.572999 74.854999 178.510001 123.265001)
+    (links 4)
+    (no_connects 4)
+    (area -1.81356 17.769679 141.031199 115.19408)
     (thickness 1.6)
     (drawings 1)
     (tracks 0)
     (zones 0)
-    (modules 0)
-    (nets 1)
+    (modules 1)
+    (nets 3)
   )
   (page USLetter)
@@
     (title "2x3 Push Terminal 3mm Pitch SMT")
     (date "17 Mar 2017")
-    (rev "1.0")
+    (rev 1.0)
     (company "All rights reserved.")
-    (comment 1 "help@browndoggadgets.com")
-    (comment 2 "http://browndoggadgets.com/")
+    (comment 1 help@browndoggadgets.com)
+    (comment 2 http://browndoggadgets.com/)
     (comment 3 "Brown Dog Gadgets")
   )
@@
   )
   (net 0 "")
+  (net 1 /1)
+  (net 2 /2)
   (net_class Default "This is the default net class."
     (clearance 0.254)
@@
     (uvia_dia 0.6858)
     (uvia_drill 0.3302)
+    (add_net /1)
+    (add_net /2)
   )
-  (gr_text "FABRICATION NOTES\n\n1. THIS IS A 2 LAYER BOARD. \n2. EXTERNAL LAYERS SHALL HAVE 1 OZ COPPER.\n3. MATERIAL: FR4 AND 0.062 INCH +/- 10% THICK.\n4. BOARDS SHALL BE ROHS COMPLIANT. \n5. MANUFACTURE IN ACCORDANCE WITH IPC-6012 CLASS 2\n6. MASK: BOTH SIDES OF THE BOARD SHALL HAVE \n   SOLDER MASK (ANY COLOR) OVER BARE COPPER. \n7. SILK: BOTH SIDES OF THE BOARD SHALL HAVE \n   WHITE SILKSCREEN. DO NOT PLACE SILK OVER BARE COPPER.\n8. FINISH: ENIG.\n9. MINIMUM TRACE WIDTH - 0.006 INCH.\n   MINIMUM SPACE - 0.006 INCH.\n   MINIMUM HOLE DIA - 0.013 INCH. \n10. MAX HOLE PLACEMENT TOLERANCE OF +/- 0.003 INCH.\n11. MAX HOLE DIAMETER TOLERANCE OF +/- 0.003 INCH AFTER PLATING." (at 120.3198 68.326) (layer Dwgs.User)
+  (module Crazy_Circuits:PUSH-TERMINAL-3MM-SMT-2x3 (layer F.Cu)
+    (at 3.95732 29.844)
+    (descr "10mm LED 5mm pitch through hole center polarized")
+    (fp_text reference J1 (at 4 -5) (layer B.SilkS) hide
+      (effects (font (size 1 1) (thickness 0.15)) (justify mirror))
+    )
+    (fp_text value "Push Terminal Block" (at 12 -4) (layer F.Fab) hide
+      (effects (font (size 1 1) (thickness 0.15)))
+    )
+    (fp_line (start 0 -7.8) (end 16.2 -7.8) (layer F.SilkS) (width 0.5))
+    (fp_text user HOLES (at 17.4 -4 90) (layer F.Fab)
+      (effects (font (size 0.762 0.762) (thickness 0.15)))
+    )
+    (fp_text user 3.5mm (at 12 -6) (layer F.Fab)
+      (effects (font (size 1 1) (thickness 0.15)))
+    )
+    (fp_text user TERMINAL (at 12 -2) (layer F.Fab)
+      (effects (font (size 1 1) (thickness 0.15)))
+    )
+    (fp_text user SCREW (at 12 -4) (layer F.Fab)
+      (effects (font (size 1 1) (thickness 0.15)))
+    )
+    (fp_line (start 8 -1.2) (end 8 -6.8) (layer F.Fab) (width 0.1))
+    (fp_line (start 16 -1.2) (end 8 -1.2) (layer F.Fab) (width 0.1))
+    (fp_line (start 16 -6.8) (end 16 -1.2) (layer F.Fab) (width 0.1))
+    (fp_line (start 8 -6.8) (end 16 -6.8) (layer F.Fab) (width 0.1))
+    (fp_text user %R (at 12 -4) (layer F.Fab) hide
+      (effects (font (size 1 1) (thickness 0.15)))
+    )
+    (fp_line (start 16 -8) (end 0 -8) (layer B.Mask) (width 7.2))
+    (fp_line (start 16 -8) (end 0 -8) (layer B.Cu) (width 7.2))
+    (fp_line (start 16 0) (end 0 0) (layer B.Mask) (width 7.2))
+    (fp_line (start 16 0) (end 0 0) (layer B.Cu) (width 7.2))
+    (fp_line (start 15.9 -11.8) (end 0.1 -11.8) (layer Edge.Cuts) (width 0.04064))
+    (fp_line (start 15.9 3.8) (end 0.1 3.8) (layer Edge.Cuts) (width 0.04064))
+    (fp_line (start 19.8 -0.1) (end 19.8 -7.9) (layer Edge.Cuts) (width 0.04064))
+    (fp_line (start -3.8 -0.1) (end -3.8 -7.9) (layer Edge.Cuts) (width 0.04064))
+    (fp_arc (start 15.9 -7.9) (end 15.9 -11.8) (angle 90) (layer Edge.Cuts) (width 0.04064))
+    (fp_arc (start 15.9 -0.1) (end 19.8 -0.1) (angle 90) (layer Edge.Cuts) (width 0.04064))
+    (fp_arc (start 0.1 -0.1) (end 0.1 3.8) (angle 90) (layer Edge.Cuts) (width 0.04064))
+    (fp_arc (start 0.1 -7.9) (end -3.8 -7.9) (angle 90) (layer Edge.Cuts) (width 0.04064))
+    (fp_line (start 15.9 -11.8) (end 0.1 -11.8) (layer F.Fab) (width 0.04064))
+    (fp_line (start 15.9 3.8) (end 0.1 3.8) (layer F.Fab) (width 0.04064))
+    (fp_line (start 19.8 -0.1) (end 19.8 -7.9) (layer F.Fab) (width 0.04064))
+    (fp_line (start -3.8 -0.1) (end -3.8 -7.9) (layer F.Fab) (width 0.04064))
+    (fp_arc (start 15.9 -7.9) (end 15.9 -11.8) (angle 90) (layer F.Fab) (width 0.04064))
+    (fp_arc (start 15.9 -0.1) (end 19.8 -0.1) (angle 90) (layer F.Fab) (width 0.04064))
+    (fp_arc (start 0.1 -0.1) (end 0.1 3.8) (angle 90) (layer F.Fab) (width 0.04064))
+    (fp_arc (start 0.1 -7.9) (end -3.8 -7.9) (angle 90) (layer F.Fab) (width 0.04064))
+    (fp_line (start 16 0) (end 0 0) (layer F.SilkS) (width 7.2))
+    (fp_line (start 9 -5.2) (end 15 -5.2) (layer F.Cu) (width 1))
+    (fp_line (start 9 -2.6) (end 15 -2.6) (layer F.Cu) (width 1))
+    (fp_text user "THIS END" (at 18.6 -4 90) (layer F.Fab)
+      (effects (font (size 0.762 0.762) (thickness 0.15)))
+    )
+    (pad 1 smd rect (at 9 -5.4 90) (size 1.4 2.5) (layers F.Cu F.Paste F.Mask)
+      (net 1 /1))
+    (pad 2 smd rect (at 9 -2.4 90) (size 1.4 2.5) (layers F.Cu F.Paste F.Mask)
+      (net 2 /2))
+    (pad 1 smd rect (at 15 -5.4 90) (size 1.4 2.5) (layers F.Cu F.Paste F.Mask)
+      (net 1 /1))
+    (pad 2 smd rect (at 15 -2.4 90) (size 1.4 2.5) (layers F.Cu F.Paste F.Mask)
+      (net 2 /2))
+    (pad - thru_hole circle (at 0 0) (size 6 6) (drill 4.98) (layers *.Cu B.Mask))
+    (pad + thru_hole circle (at 0 -8) (size 6 6) (drill 4.98) (layers *.Cu B.Mask))
+    (pad + thru_hole circle (at 16 -8) (size 6 6) (drill 4.98) (layers *.Cu B.Mask))
+    (pad - thru_hole circle (at 16 0) (size 6 6) (drill 4.98) (layers *.Cu B.Mask))
+    (pad + thru_hole circle (at 8 -8) (size 6 6) (drill 4.98) (layers *.Cu B.Mask))
+    (pad - thru_hole circle (at 8 0) (size 6 6) (drill 4.98) (layers *.Cu B.Mask))
+    (pad 1 thru_hole circle (at 12 -5.2) (size 0.762 0.762) (drill 0.3302) (layers *.Cu B.Mask)
+      (net 1 /1))
+    (pad 2 thru_hole circle (at 12 -2.6) (size 0.762 0.762) (drill 0.3302) (layers *.Cu B.Mask)
+      (net 2 /2))
+  )
+  (gr_text "FABRICATION NOTES\n\n1. THIS IS A 2 LAYER BOARD. \n2. EXTERNAL LAYERS SHALL HAVE 1 OZ COPPER.\n3. MATERIAL: FR4 AND 0.062 INCH +/- 10% THICK.\n4. BOARDS SHALL BE ROHS COMPLIANT. \n5. MANUFACTURE IN ACCORDANCE WITH IPC-6012 CLASS 2\n6. MASK: BOTH SIDES OF THE BOARD SHALL HAVE \n   SOLDER MASK (PURPLE) OVER BARE COPPER. \n7. SILK: BOTH SIDES OF THE BOARD SHALL HAVE \n   WHITE SILKSCREEN. DO NOT PLACE SILK OVER BARE COPPER.\n8. FINISH: ENIG.\n9. MINIMUM TRACE WIDTH - 0.006 INCH.\n   MINIMUM SPACE - 0.006 INCH.\n   MINIMUM HOLE DIA - 0.013 INCH. \n10. MAX HOLE PLACEMENT TOLERANCE OF +/- 0.003 INCH.\n11. MAX HOLE DIAMETER TOLERANCE OF +/- 0.003 INCH AFTER PLATING." (at -1.81356 80.52308) (layer Dwgs.User)
     (effects (font (size 2.54 2.54) (thickness 0.254)) (justify left))
   )
