File: Circuit-Kits/Modules/3x4-555-Timer-8DIP-Breakout/3x4-555-Timer-8DIP-Breakout.sch (KiCad schematic (older format))
At the start: 1 part, among them U1 555TIMER

Commit message: Port project to KiCad 5.0
Parts:
- removed U1: 555TIMER, Crazy_Circuits:DIP8-3x4-555Timer, symbol 555TIMER
- added U1: 555TIMER, Crazy_Circuits:DIP8-3x4, symbol crazy_circuits:555TIMER
Changed lines of the file:
@@
-EESchema Schematic File Version 2
+EESchema Schematic File Version 4
 LIBS:crazy_circuits
 LIBS:3x4-555-Timer-8DIP-Breakout-cache
-EELAYER 25 0
+EELAYER 26 0
 EELAYER END
 $Descr USLetter 11000 8500
@@
 Comment4 ""
 $EndDescr
-$Comp
-L 555TIMER U1
-U 1 1 5882F33F
-P 5075 3925
-F 0 "U1" H 5000 4325 50  0000 C CNN
-F 1 "555TIMER" H 5125 3525 50  0000 C CNN
-F 2 "Crazy_Circuits:DIP8-3x4-555Timer" H 4900 4225 50  0001 C CNN
-F 3 "" H 5000 4325 50  0001 C CNN
-F 4 "IC OSC 555 TIMER 8-DIP" H 5100 4425 50  0000 C CNN "Description"
-F 5 "Fairchild" H 5200 4525 50  0000 C CNN "MF_Name"
-F 6 "LM555CN" H 5300 4625 50  0000 C CNN "MF_PN"
-F 7 "Digikey" H 5400 4725 50  0000 C CNN "S1_Name"
-F 8 "LM555CNFS-ND" H 5500 4825 50  0000 C CNN "S1_PN"
-	1    5075 3925
-	1    0    0    -1
-$EndComp
 Wire Wire Line
 	5200 3675 5325 3675
@@
 Wire Wire Line
 	5200 4200 5325 4200
+$Comp
+L crazy_circuits:555TIMER U1
+U 1 1 5B84BBFB
+P 5075 3925
+F 0 "U1" H 5000 4325 50  0000 C CNN
+F 1 "555TIMER" H 5125 3525 50  0000 C CNN
+F 2 "Crazy_Circuits:DIP8-3x4" H 4900 4225 50  0001 C CNN
+F 3 "" H 5000 4325 50  0001 C CNN
+F 4 "IC OSC 555 TIMER 8-DIP" H 5100 4425 50  0001 C CNN "Description"
+F 5 "Fairchild" H 5200 4525 50  0001 C CNN "MF_Name"
+F 6 "LM555CN" H 5300 4625 50  0001 C CNN "MF_PN"
+F 7 "Digikey" H 5400 4725 50  0001 C CNN "S1_Name"
+F 8 "LM555CNFS-ND" H 5500 4825 50  0001 C CNN "S1_PN"
+	1    5075 3925
+	1    0    0    -1
+$EndComp
 $EndSCHEMATC
