File: Circuit-Kits/Modules/6x10-Feather-Bluefruit-LE/6x10-Feather-Bluefruit-LE.sch (KiCad schematic (older format))
At the start: 1 part, among them U1 ADAFRUIT-FEATHER-BLUEFRUIT-LE

Commit message: Port project to KiCad 5.0
Parts:
- U1: symbol ADAFRUIT-FEATHER-BLUEFRUIT-LE -> crazy_circuits:ADAFRUIT-FEATHER-BLUEFRUIT-LE
Connections:
- wire segments 27 -> 28
Changed lines of the file:
@@
-EESchema Schematic File Version 2
+EESchema Schematic File Version 4
 LIBS:crazy_circuits
-LIBS:6x10-Feather-Bluefruit-LE-cache
-EELAYER 25 0
+EELAYER 26 0
 EELAYER END
 $Descr USLetter 11000 8500
@@
 $EndDescr
 $Comp
-L ADAFRUIT-FEATHER-BLUEFRUIT-LE U1
+L crazy_circuits:ADAFRUIT-FEATHER-BLUEFRUIT-LE U1
 U 1 1 5A7C752E
 P 4175 3475
@@
 $EndComp
 $Comp
-L VCC #PWR01
+L crazy_circuits:VCC #PWR01
 U 1 1 5A7C75BB
 P 4625 1975
@@
 NoConn ~ 4375 2125
 $Comp
-L GND #PWR02
+L crazy_circuits:GND #PWR02
 U 1 1 5A7C898D
 P 4600 5350
@@
 Connection ~ 4625 2225
 Wire Wire Line
-	4625 1975 4625 2325
+	4625 1975 4625 2225
 Text Label 4475 2525 0    50   ~ 0
 ~RST
@@
 NoConn ~ 4375 3825
 NoConn ~ 4375 3925
+Wire Wire Line
+	4625 2225 4625 2325
 $EndSCHEMATC
