File: Circuit-Kits/Modules/5x11-Arduino-Nano-Robot-Version/5x11-Arduino-Nano-Robot-Version.sch (KiCad schematic (older format))
At the start: 6 parts, among them J1 PWM, J2 PWM, J3 PWM, J4 ANALOG, J5 ANALOG, U1 ARDUINO-NANO

Commit message: Add Arduino Nano Robot v1.1 with schematic in PDF.
Parts:
- added J6: PWR, Crazy_NonLego:CONN-HEADER-STRAIGHT-P2.54MM-1x02, symbol HEADER-MALE-2POS-TH-1x02-P0.1IN
Connections:
- net labels removed: VCC
- wire segments 54 -> 55
Changed lines of the file:
@@
-	1    0    0    -1
-$EndComp
-$Comp
-L VCC #PWR02
-U 1 1 58FE4F68
-P 3800 1150
-F 0 "#PWR02" H 3800 1000 50  0001 C CNN
-F 1 "VCC" H 3800 1300 50  0000 C CNN
-F 2 "" H 3800 1150 50  0000 C CNN
-F 3 "" H 3800 1150 50  0000 C CNN
-	1    3800 1150
 	1    0    0    -1
 $EndComp
@@
 	3800 1675 3550 1675
 Wire Wire Line
-	3725 1775 3725 3750
+	3725 1200 3725 3750
 Wire Wire Line
 	3725 3675 3550 3675
@@
 	3800 2150 3550 2150
 Wire Wire Line
-	3800 1150 3800 3575
+	3800 950  3800 3575
 Wire Wire Line
 	3800 2625 3550 2625
@@
 	4200 3550 5000 3550
 Wire Wire Line
-	5000 1100 4775 1100
+	3550 1100 5000 1100
 Wire Wire Line
 	5000 1200 4775 1200
@@
 	4625 4050 4625 4275
 $Comp
-L GND #PWR03
+L GND #PWR02
 U 1 1 58FE5E9A
 P 4625 4275
-F 0 "#PWR03" H 4625 4025 50  0001 C CNN
+F 0 "#PWR02" H 4625 4025 50  0001 C CNN
 F 1 "GND" H 4625 4125 50  0000 C CNN
 F 2 "" H 4625 4275 50  0000 C CNN
@@
 Text Label 4775 1000 0    50   ~ 0
 VIN
-Text Label 4775 1100 0    50   ~ 0
-5V
 Text Label 4775 1200 0    50   ~ 0
 3V
 Text Label 4775 1450 0    50   ~ 0
 RST
+Connection ~ 3800 1100
+$Comp
+L 5V #PWR03
+U 1 1 590DB2E6
+P 3800 950
+F 0 "#PWR03" H 3800 800 50  0001 C CNN
+F 1 "5V" H 3800 1100 50  0000 C CNN
+F 2 "" H 3800 950 50  0000 C CNN
+F 3 "" H 3800 950 50  0000 C CNN
+	1    3800 950
+	1    0    0    -1
+$EndComp
+Wire Wire Line
+	3550 1200 3725 1200
+Connection ~ 3725 1775
+$Comp
+L HEADER-MALE-2POS-TH-1x02-P0.1IN J6
+U 1 1 590DBB8D
+P 3350 1150
+F 0 "J6" H 3300 1300 50  0000 L CNN
+F 1 "PWR" H 3300 1000 50  0000 L CNN
+F 2 "Crazy_NonLego:CONN-HEADER-STRAIGHT-P2.54MM-1x02" H 3350 800 50  0001 C CIN
+F 3 "https://cdn.harwin.com/pdfs/60page140.pdf" H 3350 1150 5   0001 C CNN
+F 4 "HEADER MALE 2POS TH 1x02 0.1IN" H 3350 800 50  0001 C CIN "Description"
+F 5 "Harwin" H 3350 800 50  0001 C CIN "MF_Name"
+F 6 "M20-9990246" H 3350 800 50  0001 C CIN "MF_PN"
+F 7 "Digikey" H 3350 800 50  0001 C CIN "S1_Name"
+F 8 "952-2262-ND" H 3350 800 50  0001 C CIN "S1_PN"
+	1    3350 1150
+	-1   0    0    -1
+$EndComp
 $EndSCHEMATC

Commit message: 5x11 Arduino Nano Robot v1.5 uses A4, A5
Connections:
- net labels added: A5
- net labels removed: A3
Changed lines of the file:
@@
 $EndDescr
 $Comp
-L GND #PWR01
+L GND #PWR1
 U 1 1 58FE4F4A
 P 3725 3750
-F 0 "#PWR01" H 3725 3500 50  0001 C CNN
+F 0 "#PWR1" H 3725 3500 50  0001 C CNN
 F 1 "GND" H 3725 3600 50  0000 C CNN
 F 2 "" H 3725 3750 50  0000 C CNN
@@
 D6
 Text Label 3875 3000 0    50   ~ 0
-A3
+A4
 Text Label 3875 3475 0    50   ~ 0
-A4
+A5
 $Comp
 L HEADER-MALE-3POS-TH-1x03-P0.1IN J1
@@
 	-1   0    0    -1
 $EndComp
-Wire Wire Line
-	3550 1575 4550 1575
-Wire Wire Line
-	3800 1675 3550 1675
-Wire Wire Line
-	3725 1200 3725 3750
-Wire Wire Line
-	3725 3675 3550 3675
-Wire Wire Line
-	3550 3200 3725 3200
-Connection ~ 3725 3675
-Wire Wire Line
-	3725 2725 3550 2725
-Connection ~ 3725 3200
-Wire Wire Line
-	3725 2250 3550 2250
-Connection ~ 3725 2725
-Wire Wire Line
-	3550 1775 3725 1775
-Connection ~ 3725 2250
-Wire Wire Line
-	3800 2150 3550 2150
-Wire Wire Line
-	3800 950  3800 3575
-Wire Wire Line
-	3800 2625 3550 2625
-Connection ~ 3800 2150
-Wire Wire Line
-	3800 3100 3550 3100
-Connection ~ 3800 2625
-Wire Wire Line
-	3800 3575 3550 3575
-Connection ~ 3800 3100
-Wire Wire Line
-	3550 2050 4550 2050
-Wire Wire Line
-	3550 2525 4550 2525
-Wire Wire Line
-	3550 3000 4550 3000
-Wire Wire Line
-	3550 3475 4200 3475
-Connection ~ 3800 1675
-Wire Wire Line
-	5000 1000 4775 1000
-Wire Wire Line
-	4550 1575 4550 2000
-Wire Wire Line
-	4550 2000 5000 2000
-Wire Wire Line
-	4550 2050 4550 2200
-Wire Wire Line
-	4550 2200 5000 2200
-Wire Wire Line
-	4550 2525 4550 2300
-Wire Wire Line
-	4550 2300 5000 2300
-Wire Wire Line
-	4550 3000 4550 3450
-Wire Wire Line
-	4550 3450 5000 3450
-Wire Wire Line
-	4200 3475 4200 3550
-Wire Wire Line
-	4200 3550 5000 3550
-Wire Wire Line
-	3550 1100 5000 1100
-Wire Wire Line
-	5000 1200 4775 1200
-Wire Wire Line
-	3800 1300 5000 1300
-Wire Wire Line
-	4775 1450 5000 1450
-Wire Wire Line
-	4950 1550 5000 1550
-Wire Wire Line
-	4950 1450 4950 1550
-Connection ~ 4950 1450
-Wire Wire Line
-	5000 1700 4775 1700
-Wire Wire Line
-	4775 1800 5000 1800
-Wire Wire Line
-	5000 1900 4775 1900
-Wire Wire Line
-	5000 2100 4775 2100
-Wire Wire Line
-	5000 2400 4775 2400
-Wire Wire Line
-	4775 2500 5000 2500
-Wire Wire Line
-	5000 2600 4775 2600
-Wire Wire Line
-	4775 2700 5000 2700
-Wire Wire Line
-	5000 2800 4775 2800
-Wire Wire Line
-	4775 2900 5000 2900
-Wire Wire Line
-	5000 3000 4775 3000
-Wire Wire Line
-	5000 3150 4775 3150
-Wire Wire Line
-	4775 3250 5000 3250
-Wire Wire Line
-	5000 3350 4775 3350
-Wire Wire Line
-	5000 3650 4775 3650
-Wire Wire Line
-	4775 3750 5000 3750
-Wire Wire Line
-	5000 3850 4775 3850
-Wire Wire Line
-	4625 4050 5000 4050
-Wire Wire Line
-	4625 4150 5000 4150
-Wire Wire Line
-	4625 4050 4625 4275
-$Comp
-L GND #PWR02
+$Comp
+L GND #PWR3
 U 1 1 58FE5E9A
 P 4625 4275
-F 0 "#PWR02" H 4625 4025 50  0001 C CNN
+F 0 "#PWR3" H 4625 4025 50  0001 C CNN
 F 1 "GND" H 4625 4125 50  0000 C CNN
 F 2 "" H 4625 4275 50  0000 C CNN
@@
 	1    0    0    -1
 $EndComp
-Connection ~ 4625 4150
-Connection ~ 3800 1300
 Text Label 4775 1000 0    50   ~ 0
 VIN
@@
 Text Label 4775 1450 0    50   ~ 0
 RST
-Connection ~ 3800 1100
-$Comp
-L 5V #PWR03
+$Comp
+L 5V #PWR2
 U 1 1 590DB2E6
 P 3800 950
-F 0 "#PWR03" H 3800 800 50  0001 C CNN
+F 0 "#PWR2" H 3800 800 50  0001 C CNN
 F 1 "5V" H 3800 1100 50  0000 C CNN
 F 2 "" H 3800 950 50  0000 C CNN
@@
 	1    0    0    -1
 $EndComp
-Wire Wire Line
-	3550 1200 3725 1200
-Connection ~ 3725 1775
 $Comp
 L HEADER-MALE-2POS-TH-1x02-P0.1IN J6
@@
 	-1   0    0    -1
 $EndComp
+Wire Wire Line
+	3550 1575 4550 1575
+Wire Wire Line
+	3800 1675 3550 1675
+Wire Wire Line
+	3725 1200 3725 3750
+Wire Wire Line
+	3725 3675 3550 3675
+Wire Wire Line
+	3550 3200 3725 3200
+Connection ~ 3725 3675
+Wire Wire Line
+	3725 2725 3550 2725
+Connection ~ 3725 3200
+Wire Wire Line
+	3725 2250 3550 2250
+Connection ~ 3725 2725
+Wire Wire Line
+	3550 1775 3725 1775
+Connection ~ 3725 2250
+Wire Wire Line
+	3800 2150 3550 2150
+Wire Wire Line
+	3800 950  3800 3575
+Wire Wire Line
+	3800 2625 3550 2625
+Connection ~ 3800 2150
+Wire Wire Line
+	3800 3100 3550 3100
+Connection ~ 3800 2625
+Wire Wire Line
+	3800 3575 3550 3575
+Connection ~ 3800 3100
+Wire Wire Line
+	3550 2050 4550 2050
+Wire Wire Line
+	3550 2525 4550 2525
+Wire Wire Line
+	3550 3000 4550 3000
+Wire Wire Line
+	3550 3475 4200 3475
+Connection ~ 3800 1675
+Wire Wire Line
+	5000 1000 4775 1000
+Wire Wire Line
+	4550 1575 4550 2000
+Wire Wire Line
+	4550 2000 5000 2000
+Wire Wire Line
+	4550 2050 4550 2200
+Wire Wire Line
+	4550 2200 5000 2200
+Wire Wire Line
+	4550 2525 4550 2300
+Wire Wire Line
+	4550 2300 5000 2300
+Wire Wire Line
+	4550 3000 4550 3550
+Wire Wire Line
+	4200 3475 4200 3650
+Wire Wire Line
+	3550 1100 5000 1100
+Wire Wire Line
+	5000 1200 4775 1200
+Wire Wire Line
+	3800 1300 5000 1300
+Wire Wire Line
+	4775 1450 5000 1450
+Wire Wire Line
+	4950 1550 5000 1550
+Wire Wire Line
+	4950 1450 4950 1550
+Connection ~ 4950 1450
+Wire Wire Line
+	5000 1700 4775 1700
+Wire Wire Line
+	4775 1800 5000 1800
+Wire Wire Line
+	5000 1900 4775 1900
+Wire Wire Line
+	5000 2100 4775 2100
+Wire Wire Line
+	5000 2400 4775 2400
+Wire Wire Line
+	4775 2500 5000 2500
+Wire Wire Line
+	5000 2600 4775 2600
+Wire Wire Line
+	4775 2700 5000 2700
+Wire Wire Line
+	5000 2800 4775 2800
+Wire Wire Line
+	4775 2900 5000 2900
+Wire Wire Line
+	5000 3000 4775 3000
+Wire Wire Line
+	5000 3150 4775 3150
+Wire Wire Line
+	4775 3250 5000 3250
+Wire Wire Line
+	5000 3350 4775 3350
+Wire Wire Line
+	4200 3650 5000 3650
+Wire Wire Line
+	4775 3750 5000 3750
+Wire Wire Line
+	5000 3850 4775 3850
+Wire Wire Line
+	4625 4050 5000 4050
+Wire Wire Line
+	4625 4150 5000 4150
+Wire Wire Line
+	4625 4050 4625 4275
+Connection ~ 4625 4150
+Connection ~ 3800 1300
+Connection ~ 3800 1100
+Wire Wire Line
+	3550 1200 3725 1200
+Connection ~ 3725 1775
+Wire Wire Line
+	4550 3550 5000 3550
+Wire Wire Line
+	5000 3450 4775 3450
 $EndSCHEMATC

Commit message: Adjust headers. Release 5x11 Ardu Nano Robot v1.6.
Parts:
- removed J6: PWR, Crazy_NonLego:CONN-HEADER-STRAIGHT-P2.54MM-1x02, symbol HEADER-MALE-2POS-TH-1x02-P0.1IN
- added J4: PWM, Crazy_NonLego:CONN-HEADER-STRAIGHT-P2.54MM-1x03, symbol HEADER-MALE-3POS-TH-1x03-P0.1IN
- J1, J2, J3: MF_PN M20-9992046 -> M20-9990346; S1_PN 952-1902-ND -> 952-2264-ND
- J5: renamed from J4; MF_PN M20-9992046 -> M20-9990346; S1_PN 952-1902-ND -> 952-2264-ND
- J6: renamed from J5; MF_PN M20-9992046 -> M20-9990346; S1_PN 952-1902-ND -> 952-2264-ND
Connections:
- net labels added: D9
- wire segments 55 -> 58
Other:
- moved on the sheet: J5, J6
Changed lines of the file:
@@
 L GND #PWR1
 U 1 1 58FE4F4A
-P 3725 3750
-F 0 "#PWR1" H 3725 3500 50  0001 C CNN
-F 1 "GND" H 3725 3600 50  0000 C CNN
-F 2 "" H 3725 3750 50  0000 C CNN
-F 3 "" H 3725 3750 50  0000 C CNN
-	1    3725 3750
+P 3725 4225
+F 0 "#PWR1" H 3725 3975 50  0001 C CNN
+F 1 "GND" H 3725 4075 50  0000 C CNN
+F 2 "" H 3725 4225 50  0000 C CNN
+F 3 "" H 3725 4225 50  0000 C CNN
+	1    3725 4225
 	1    0    0    -1
 $EndComp
@@
 Text Label 3875 2525 0    50   ~ 0
 D6
-Text Label 3875 3000 0    50   ~ 0
+Text Label 3875 3475 0    50   ~ 0
 A4
-Text Label 3875 3475 0    50   ~ 0
+Text Label 3875 3950 0    50   ~ 0
 A5
 $Comp
@@
 F 4 "HEADER MALE 3POS TH 1x03 0.1IN" H 3350 1325 50  0001 C CIN "Description"
 F 5 "Harwin" H 3350 1325 50  0001 C CIN "MF_Name"
-F 6 "M20-9992046" H 3350 1325 50  0001 C CIN "MF_PN"
+F 6 "M20-9990346" H 3350 1325 50  0001 C CIN "MF_PN"
 F 7 "Digikey" H 3350 1325 50  0001 C CIN "S1_Name"
-F 8 "952-1902-ND" H 3350 1325 50  0001 C CIN "S1_PN"
+F 8 "952-2264-ND" H 3350 1325 50  0001 C CIN "S1_PN"
 	1    3350 1675
 	-1   0    0    -1
 $EndComp
 $Comp
-L HEADER-MALE-3POS-TH-1x03-P0.1IN J2
-U 1 1 58FE541D
-P 3350 2150
-F 0 "J2" H 3300 2350 50  0000 L CNN
-F 1 "PWM" H 3300 1950 50  0000 L CNN
-F 2 "Crazy_NonLego:CONN-HEADER-STRAIGHT-P2.54MM-1x03" H 3350 1800 50  0001 C CIN
-F 3 "https://cdn.harwin.com/pdfs/60page140.pdf" H 3350 2150 5   0001 C CNN
-F 4 "HEADER MALE 3POS TH 1x03 0.1IN" H 3350 1800 50  0001 C CIN "Description"
-F 5 "Harwin" H 3350 1800 50  0001 C CIN "MF_Name"
-F 6 "M20-9992046" H 3350 1800 50  0001 C CIN "MF_PN"
-F 7 "Digikey" H 3350 1800 50  0001 C CIN "S1_Name"
-F 8 "952-1902-ND" H 3350 1800 50  0001 C CIN "S1_PN"
-	1    3350 2150
-	-1   0    0    -1
-$EndComp
-$Comp
-L HEADER-MALE-3POS-TH-1x03-P0.1IN J3
-U 1 1 58FE5461
-P 3350 2625
-F 0 "J3" H 3300 2825 50  0000 L CNN
-F 1 "PWM" H 3300 2425 50  0000 L CNN
-F 2 "Crazy_NonLego:CONN-HEADER-STRAIGHT-P2.54MM-1x03" H 3350 2275 50  0001 C CIN
-F 3 "https://cdn.harwin.com/pdfs/60page140.pdf" H 3350 2625 5   0001 C CNN
-F 4 "HEADER MALE 3POS TH 1x03 0.1IN" H 3350 2275 50  0001 C CIN "Description"
-F 5 "Harwin" H 3350 2275 50  0001 C CIN "MF_Name"
-F 6 "M20-9992046" H 3350 2275 50  0001 C CIN "MF_PN"
-F 7 "Digikey" H 3350 2275 50  0001 C CIN "S1_Name"
-F 8 "952-1902-ND" H 3350 2275 50  0001 C CIN "S1_PN"
-	1    3350 2625
-	-1   0    0    -1
-$EndComp
-$Comp
-L HEADER-MALE-3POS-TH-1x03-P0.1IN J4
+L HEADER-MALE-3POS-TH-1x03-P0.1IN J5
 U 1 1 58FE54AA
-P 3350 3100
-F 0 "J4" H 3300 3300 50  0000 L CNN
-F 1 "ANALOG" H 3300 2900 50  0000 L CNN
-F 2 "Crazy_NonLego:CONN-HEADER-STRAIGHT-P2.54MM-1x03" H 3350 2750 50  0001 C CIN
-F 3 "https://cdn.harwin.com/pdfs/60page140.pdf" H 3350 3100 5   0001 C CNN
-F 4 "HEADER MALE 3POS TH 1x03 0.1IN" H 3350 2750 50  0001 C CIN "Description"
-F 5 "Harwin" H 3350 2750 50  0001 C CIN "MF_Name"
-F 6 "M20-9992046" H 3350 2750 50  0001 C CIN "MF_PN"
-F 7 "Digikey" H 3350 2750 50  0001 C CIN "S1_Name"
-F 8 "952-1902-ND" H 3350 2750 50  0001 C CIN "S1_PN"
-	1    3350 3100
-	-1   0    0    -1
-$EndComp
-$Comp
-L HEADER-MALE-3POS-TH-1x03-P0.1IN J5
-U 1 1 58FE54F2
 P 3350 3575
 F 0 "J5" H 3300 3775 50  0000 L CNN
@@
 F 4 "HEADER MALE 3POS TH 1x03 0.1IN" H 3350 3225 50  0001 C CIN "Description"
 F 5 "Harwin" H 3350 3225 50  0001 C CIN "MF_Name"
-F 6 "M20-9992046" H 3350 3225 50  0001 C CIN "MF_PN"
+F 6 "M20-9990346" H 3350 3225 50  0001 C CIN "MF_PN"
 F 7 "Digikey" H 3350 3225 50  0001 C CIN "S1_Name"
-F 8 "952-1902-ND" H 3350 3225 50  0001 C CIN "S1_PN"
+F 8 "952-2264-ND" H 3350 3225 50  0001 C CIN "S1_PN"
 	1    3350 3575
+	-1   0    0    -1
+$EndComp
+$Comp
+L HEADER-MALE-3POS-TH-1x03-P0.1IN J6
+U 1 1 58FE54F2
+P 3350 4050
+F 0 "J6" H 3300 4250 50  0000 L CNN
+F 1 "ANALOG" H 3300 3850 50  0000 L CNN
+F 2 "Crazy_NonLego:CONN-HEADER-STRAIGHT-P2.54MM-1x03" H 3350 3700 50  0001 C CIN
+F 3 "https://cdn.harwin.com/pdfs/60page140.pdf" H 3350 4050 5   0001 C CNN
+F 4 "HEADER MALE 3POS TH 1x03 0.1IN" H 3350 3700 50  0001 C CIN "Description"
+F 5 "Harwin" H 3350 3700 50  0001 C CIN "MF_Name"
+F 6 "M20-9990346" H 3350 3700 50  0001 C CIN "MF_PN"
+F 7 "Digikey" H 3350 3700 50  0001 C CIN "S1_Name"
+F 8 "952-2264-ND" H 3350 3700 50  0001 C CIN "S1_PN"
+	1    3350 4050
 	-1   0    0    -1
 $EndComp
@@
 	1    0    0    -1
 $EndComp
-$Comp
-L HEADER-MALE-2POS-TH-1x02-P0.1IN J6
-U 1 1 590DBB8D
-P 3350 1150
-F 0 "J6" H 3300 1300 50  0000 L CNN
-F 1 "PWR" H 3300 1000 50  0000 L CNN
-F 2 "Crazy_NonLego:CONN-HEADER-STRAIGHT-P2.54MM-1x02" H 3350 800 50  0001 C CIN
-F 3 "https://cdn.harwin.com/pdfs/60page140.pdf" H 3350 1150 5   0001 C CNN
-F 4 "HEADER MALE 2POS TH 1x02 0.1IN" H 3350 800 50  0001 C CIN "Description"
-F 5 "Harwin" H 3350 800 50  0001 C CIN "MF_Name"
-F 6 "M20-9990246" H 3350 800 50  0001 C CIN "MF_PN"
-F 7 "Digikey" H 3350 800 50  0001 C CIN "S1_Name"
-F 8 "952-2262-ND" H 3350 800 50  0001 C CIN "S1_PN"
-	1    3350 1150
-	-1   0    0    -1
-$EndComp
 Wire Wire Line
 	3550 1575 4550 1575
@@
 	3800 1675 3550 1675
 Wire Wire Line
-	3725 1200 3725 3750
-Wire Wire Line
-	3725 3675 3550 3675
-Wire Wire Line
-	3550 3200 3725 3200
+	3725 4150 3550 4150
+Wire Wire Line
+	3550 3675 3725 3675
+Connection ~ 3725 4150
+Wire Wire Line
+	3725 2725 3550 2725
 Connection ~ 3725 3675
-Wire Wire Line
-	3725 2725 3550 2725
-Connection ~ 3725 3200
 Wire Wire Line
 	3725 2250 3550 2250
@@
 	3800 2150 3550 2150
 Wire Wire Line
-	3800 950  3800 3575
+	3800 950  3800 4050
 Wire Wire Line
 	3800 2625 3550 2625
 Connection ~ 3800 2150
 Wire Wire Line
-	3800 3100 3550 3100
+	3800 3575 3550 3575
 Connection ~ 3800 2625
 Wire Wire Line
-	3800 3575 3550 3575
-Connection ~ 3800 3100
+	3800 4050 3550 4050
+Connection ~ 3800 3575
 Wire Wire Line
 	3550 2050 4550 2050
@@
 	3550 2525 4550 2525
 Wire Wire Line
-	3550 3000 4550 3000
-Wire Wire Line
 	3550 3475 4200 3475
+Wire Wire Line
+	3550 3950 4200 3950
 Connection ~ 3800 1675
 Wire Wire Line
@@
 	4550 2300 5000 2300
 Wire Wire Line
-	4550 3000 4550 3550
-Wire Wire Line
-	4200 3475 4200 3650
-Wire Wire Line
-	3550 1100 5000 1100
+	3800 1100 5000 1100
 Wire Wire Line
 	5000 1200 4775 1200
@@
 	4775 2500 5000 2500
 Wire Wire Line
-	5000 2600 4775 2600
+	4550 2600 5000 2600
 Wire Wire Line
 	4775 2700 5000 2700
@@
 Connection ~ 4625 4150
 Connection ~ 3800 1300
+Wire Wire Line
+	4200 3550 5000 3550
+Wire Wire Line
+	5000 3450 4775 3450
+Wire Wire Line
+	4200 3475 4200 3550
+Wire Wire Line
+	4200 3950 4200 3650
 Connection ~ 3800 1100
 Wire Wire Line
-	3550 1200 3725 1200
-Connection ~ 3725 1775
-Wire Wire Line
-	4550 3550 5000 3550
-Wire Wire Line
-	5000 3450 4775 3450
+	3725 1775 3725 4225
+Wire Wire Line
+	3550 3000 4550 3000
+Wire Wire Line
+	4550 3000 4550 2600
+Wire Wire Line
+	3550 3100 3800 3100
+Connection ~ 3800 3100
+Wire Wire Line
+	3550 3200 3725 3200
+Connection ~ 3725 3200
+Text Label 3875 3000 0    50   ~ 0
+D9
+$Comp
+L HEADER-MALE-3POS-TH-1x03-P0.1IN J2
+U 1 1 5AF1C185
+P 3350 2150
+F 0 "J2" H 3300 2350 50  0000 L CNN
+F 1 "PWM" H 3300 1950 50  0000 L CNN
+F 2 "Crazy_NonLego:CONN-HEADER-STRAIGHT-P2.54MM-1x03" H 3350 1800 50  0001 C CIN
+F 3 "https://cdn.harwin.com/pdfs/60page140.pdf" H 3350 2150 5   0001 C CNN
+F 4 "HEADER MALE 3POS TH 1x03 0.1IN" H 3350 1800 50  0001 C CIN "Description"
+F 5 "Harwin" H 3350 1800 50  0001 C CIN "MF_Name"
+F 6 "M20-9990346" H 3350 1800 50  0001 C CIN "MF_PN"
+F 7 "Digikey" H 3350 1800 50  0001 C CIN "S1_Name"
+F 8 "952-2264-ND" H 3350 1800 50  0001 C CIN "S1_PN"
+	1    3350 2150
+	-1   0    0    -1
+$EndComp
+$Comp
+L HEADER-MALE-3POS-TH-1x03-P0.1IN J3
+U 1 1 5AF1C1CE
+P 3350 2625
+F 0 "J3" H 3300 2825 50  0000 L CNN
+F 1 "PWM" H 3300 2425 50  0000 L CNN
+F 2 "Crazy_NonLego:CONN-HEADER-STRAIGHT-P2.54MM-1x03" H 3350 2275 50  0001 C CIN
+F 3 "https://cdn.harwin.com/pdfs/60page140.pdf" H 3350 2625 5   0001 C CNN
+F 4 "HEADER MALE 3POS TH 1x03 0.1IN" H 3350 2275 50  0001 C CIN "Description"
+F 5 "Harwin" H 3350 2275 50  0001 C CIN "MF_Name"
+F 6 "M20-9990346" H 3350 2275 50  0001 C CIN "MF_PN"
+F 7 "Digikey" H 3350 2275 50  0001 C CIN "S1_Name"
+F 8 "952-2264-ND" H 3350 2275 50  0001 C CIN "S1_PN"
+	1    3350 2625
+	-1   0    0    -1
+$EndComp
+$Comp
+L HEADER-MALE-3POS-TH-1x03-P0.1IN J4
+U 1 1 5AF1C230
+P 3350 3100
+F 0 "J4" H 3300 3300 50  0000 L CNN
+F 1 "PWM" H 3300 2900 50  0000 L CNN
+F 2 "Crazy_NonLego:CONN-HEADER-STRAIGHT-P2.54MM-1x03" H 3350 2750 50  0001 C CIN
+F 3 "https://cdn.harwin.com/pdfs/60page140.pdf" H 3350 3100 5   0001 C CNN
+F 4 "HEADER MALE 3POS TH 1x03 0.1IN" H 3350 2750 50  0001 C CIN "Description"
+F 5 "Harwin" H 3350 2750 50  0001 C CIN "MF_Name"
+F 6 "M20-9990346" H 3350 2750 50  0001 C CIN "MF_PN"
+F 7 "Digikey" H 3350 2750 50  0001 C CIN "S1_Name"
+F 8 "952-2264-ND" H 3350 2750 50  0001 C CIN "S1_PN"
+	1    3350 3100
+	-1   0    0    -1
+$EndComp
 $EndSCHEMATC
