File: Circuit-Kits/Modules/1x2-LED-1206-SMT/1x2-LED-1206-SMT.sch (KiCad schematic (older format))
At the start: 1 part

Commit message: Port project to KiCad 5.0
Parts:
- LED1: symbol LED -> crazy_circuits:LED
Changed lines of the file:
@@
 $EndDescr
 $Comp
-L LED LED1
+L crazy_circuits:LED LED1
 U 1 1 5890E035
 P 4700 4325
@@
 $EndComp
 $Comp
-L VCC #PWR?
+L crazy_circuits:VCC #PWR?
 U 1 1 5890E052
 P 4700 4075
@@
 	4700 4425 4700 4575
 $Comp
-L GND #PWR?
+L crazy_circuits:GND #PWR?
 U 1 1 5890E070
 P 4700 4575
