File: Circuit-Kits/Modules/2x2-12mm-Square-SMT-Pushbutton/2x2-12mm-Square-SMT-Pushbutton.sch (KiCad schematic (older format))
At the start: 1 part, among them SW1 B3FS-4002P

Commit message: Port project to KiCad 5.0
Parts:
- SW1: symbol SWITCH-MOMENT-SPDT-SMT-B3FS-4002P -> crazy_circuits:SWITCH-MOMENT-SPDT-SMT-B3FS-4002P
Connections:
- wire segments 6 -> 8
Changed lines of the file:
@@
-EESchema Schematic File Version 2
+EESchema Schematic File Version 4
 LIBS:crazy_circuits
-EELAYER 25 0
+EELAYER 26 0
 EELAYER END
 $Descr USLetter 11000 8500
@@
 $EndDescr
 $Comp
-L SWITCH-MOMENT-SPDT-SMT-B3FS-4002P SW1
+L crazy_circuits:SWITCH-MOMENT-SPDT-SMT-B3FS-4002P SW1
 U 1 1 5877E7CA
 P 4875 3625
@@
 	4525 3725 4525 3625
 Wire Wire Line
-	4400 3625 4575 3625
+	4400 3625 4525 3625
 Connection ~ 4525 3625
 Text Label 4400 3625 0    50   ~ 0
 1
 Wire Wire Line
-	5175 3625 5325 3625
+	5175 3625 5225 3625
 Wire Wire Line
 	5175 3725 5225 3725
@@
 Text Label 5325 3625 2    50   ~ 0
 2
+Wire Wire Line
+	4525 3625 4575 3625
+Wire Wire Line
+	5225 3625 5325 3625
 $EndSCHEMATC
