File: Circuit-Kits/Modules/2x2-LED-WHITE-SMT-LIMITED/2x2-LED-WHITE-SMT-LIMITED.sch (KiCad schematic (older format))
At the start: 2 parts

Commit message: Port project to KiCad 5.0
Parts:
- LED1: symbol LED-WHITE-1206-SMT-QBLP650-IW -> crazy_circuits:LED-WHITE-1206-SMT-QBLP650-IW
- R1: symbol RES-100-1%-1/4W-1206 -> crazy_circuits:RES-100-1%-1/4W-1206
Changed lines of the file:
@@
-EESchema Schematic File Version 2
-LIBS:crazy_circuits
-EELAYER 25 0
+EESchema Schematic File Version 4
+EELAYER 26 0
 EELAYER END
 $Descr USLetter 11000 8500
@@
 $EndDescr
 $Comp
-L VCC #PWR1
+L crazy_circuits:VCC #PWR1
 U 1 1 5AF330D8
 P 4400 3275
@@
 $EndComp
 $Comp
-L RES-100-1%-1/4W-1206 R1
+L crazy_circuits:RES-100-1%-1/4W-1206 R1
 U 1 1 5AF330EC
 P 4400 3475
@@
 $EndComp
 $Comp
-L LED-WHITE-1206-SMT-QBLP650-IW LED1
+L crazy_circuits:LED-WHITE-1206-SMT-QBLP650-IW LED1
 U 1 1 5AF3312A
 P 4400 3775
@@
 $EndComp
 $Comp
-L GND #PWR2
+L crazy_circuits:GND #PWR2
 U 1 1 5AF33182
 P 4400 3975
