File: Circuit-Kits/Modules/2x2-LED-YELLOW-SMT-LIMITED/2x2-LED-YELLOW-SMT-LIMITED.sch (KiCad schematic (older format))
At the start: 2 parts

Commit message: Port project to KiCad 5.0
Parts:
- LED1: symbol LED-YELLOW-1206-SMT-150120YS75000 -> crazy_circuits:LED-YELLOW-1206-SMT-150120YS75000
- R1: symbol RES-100-1%-1/4W-1206 -> crazy_circuits:RES-100-1%-1/4W-1206
Changed lines of the file:
@@
-EESchema Schematic File Version 2
+EESchema Schematic File Version 4
 LIBS:crazy_circuits
-EELAYER 25 0
+EELAYER 26 0
 EELAYER END
 $Descr USLetter 11000 8500
@@
 $EndDescr
 $Comp
-L VCC #PWR1
+L crazy_circuits:VCC #PWR1
 U 1 1 5AF32EF0
 P 4625 3475
@@
 $EndComp
 $Comp
-L RES-100-1%-1/4W-1206 R1
+L crazy_circuits:RES-100-1%-1/4W-1206 R1
 U 1 1 5AF32F04
 P 4625 3625
@@
 $EndComp
 $Comp
-L LED-YELLOW-1206-SMT-150120YS75000 LED1
+L crazy_circuits:LED-YELLOW-1206-SMT-150120YS75000 LED1
 U 1 1 5AF32F4A
 P 4625 3925
@@
 $EndComp
 $Comp
-L GND #PWR2
+L crazy_circuits:GND #PWR2
 U 1 1 5AF32FA2
 P 4625 4125
