File: Circuit-Kits/Modules/2x2-Tilt-Switch-SW-520D-TH/2x2-Tilt-Switch-SW-520D-TH.sch (KiCad schematic (older format))
At the start: 1 part, among them SW1 SW_TILT

Commit message: Port project to KiCad 5.0
Parts:
- SW1: symbol SW_TOGGLE -> crazy_circuits:SW_TOGGLE
Changed lines of the file:
@@
-EESchema Schematic File Version 2
+EESchema Schematic File Version 4
 LIBS:crazy_circuits
-EELAYER 25 0
+EELAYER 26 0
 EELAYER END
 $Descr USLetter 11000 8500
@@
 1
 $Comp
-L SW_TOGGLE SW1
+L crazy_circuits:SW_TOGGLE SW1
 U 1 1 58CABBD1
 P 4875 3950
@@
 F 1 "SW_TILT" H 4875 3870 50  0000 C CNN
 F 2 "Crazy_Circuits:TILT-SENSOR-SW-520D-TH-2x2" H 4875 3950 50  0001 C CNN
-F 3 "http://funduino.de/DL/SW-520D.pdf" H 4925 3675 50  0000 C CNN
+F 3 "http://funduino.de/DL/SW-520D.pdf" H 4925 3675 50  0001 C CNN
 F 4 "TILT SENSOR ROLLING BALL SW-520D" H 4875 3950 60  0001 C CNN "Description"
 F 5 "Bailin Electronics" H 4875 3950 60  0001 C CNN "MF_Name"
