File: Circuit-Kits/Modules/2x3-LED-RGB-NeoPixel-SMT/2x3-LED-RGB-NeoPixel-SMT.sch (KiCad schematic (older format))
At the start: 3 parts

Commit message: Port project to KiCad 5.0
Parts:
- C1: symbol CAP-CER-0.1UF-100V-X7R-0603 -> crazy_circuits:CAP-CER-0.1UF-16V-X7R-0603; Description CAP CER 0.1UF 100V X7R 0603 -> CAP CER 0.1UF 16V X7R 0603; MF_PN GRM188R72A104KA35D -> GCM188R71C104KA37D; S1_PN 490-3285-1-ND -> 490-4774-1-ND; Type (none) -> smt; XSize_mils (none) -> 114; YSize_mils (none) -> 59
- LED1: symbol LED-RGB-WS2812B-4SMD -> crazy_circuits:LED-RGB-WS2812B-4SMD; Package RGBLED5050 -> (none); Type (none) -> smt; Verified Not Verified -> (none)
- R1: symbol RES-470-5%-1/4W-0603 -> crazy_circuits:RES-470-5%-1_4W-0603; Package 0603 -> (none); Type (none) -> smt; Verified Not Verified -> (none)
Connections:
- wire segments 10 -> 12
Changed lines of the file:
@@
-EESchema Schematic File Version 2
+EESchema Schematic File Version 4
 LIBS:crazy_circuits
 LIBS:wickerlib
 LIBS:2x3-LED-RGB-NeoPixel-SMT-cache
-EELAYER 25 0
+EELAYER 26 0
 EELAYER END
 $Descr USLetter 11000 8500
@@
 $EndDescr
 Wire Wire Line
-	4200 3775 5050 3775
+	4200 3775 4325 3775
 Wire Wire Line
 	6050 4175 6400 4175
 Wire Wire Line
-	5550 4425 5550 4700
+	5550 4425 5550 4625
 Text Label 4600 3775 0    60   ~ 0
 VCC
@@
 Connection ~ 5550 4625
 $Comp
-L GND #PWR01
+L crazy_circuits:GND #PWR01
 U 1 1 57C8B8D5
 P 5550 4700
@@
 $EndComp
 $Comp
-L RES-470-5%-1/4W-0603 R1
+L crazy_circuits:RES-470-5%-1_4W-0603 R1
 U 1 1 57C8BA02
 P 4825 4350
@@
 F 2 "" H 4825 4000 50  0001 C CIN
 F 3 "http://rohmfs.rohm.com/en/products/databook/datasheet/passive/resistor/chip_resistor/esr.pdf" H 4825 4350 5   0001 C CNN
-F 4 "0603" H 4825 4000 50  0001 C CIN "Package"
+F 4 "RES SMD 470 OHM 5% 1/4W 0603" H 4825 4000 50  0001 C CIN "Description"
 F 5 "Rohm Semi" H 4825 4000 50  0001 C CIN "MF_Name"
 F 6 "ESR03EZPJ471" H 4825 4000 50  0001 C CIN "MF_PN"
 F 7 "Digikey" H 4825 4000 50  0001 C CIN "S1_Name"
 F 8 "RHM470DCT-ND" H 4825 4000 50  0001 C CIN "S1_PN"
-F 9 "RES SMD 470 OHM 5% 1/4W 0603" H 4825 4000 50  0001 C CIN "Description"
-F 10 "Not Verified" H 4825 4000 50  0001 C CIN "Verified"
+F 9 "smt" H 0   0   50  0001 C CNN "Type"
 	1    4825 4350
 	1    0    0    -1
@@
 Strongly recommended to place \na 100nF capacitor between VCC\nand GND between micro and pixels.
 $Comp
-L LED-RGB-WS2812B-4SMD LED1
+L crazy_circuits:LED-RGB-WS2812B-4SMD LED1
 U 1 1 57C8DCCA
 P 5500 3925
@@
 F 2 "Crazy_Circuits:LED-RGB-5050-NEOPIXEL-ROTATED-2x3" H 5500 3575 50  0001 C CIN
 F 3 "http://www.adafruit.com/datasheets/WS2812B.pdf" H 5500 3925 5   0001 C CNN
-F 4 "RGBLED5050" H 5500 3575 50  0001 C CIN "Package"
+F 4 "LED RGB WS2812B W/DVR 4SMD" H 5500 3575 50  0001 C CIN "Description"
 F 5 "Adafruit" H 5500 3575 50  0001 C CIN "MF_Name"
 F 6 "1655" H 5500 3575 50  0001 C CIN "MF_PN"
 F 7 "Digikey" H 5500 3575 50  0001 C CIN "S1_Name"
 F 8 "1528-1104-ND" H 5500 3575 50  0001 C CIN "S1_PN"
-F 9 "LED RGB WS2812B W/DVR 4SMD" H 5500 3575 50  0001 C CIN "Description"
-F 10 "Not Verified" H 5500 3575 50  0001 C CIN "Verified"
+F 9 "smt" H 0   0   50  0001 C CNN "Type"
 	1    5500 3925
 	1    0    0    -1
@@
 Connection ~ 4325 3775
 $Comp
-L GND #PWR02
+L crazy_circuits:GND #PWR02
 U 1 1 5961C601
 P 4325 4125
@@
 	4325 4125 4325 4075
 $Comp
-L CAP-CER-0.1UF-100V-X7R-0603 C1
+L crazy_circuits:CAP-CER-0.1UF-16V-X7R-0603 C1
 U 1 1 5AF9A904
 P 4325 3975
@@
 F 2 "" H 4325 3625 50  0001 C CIN
 F 3 "http://search.murata.co.jp/Ceramy/image/img/A01X/partnumbering_e_01.pdf" H 4325 3975 5   0001 C CNN
-F 4 "CAP CER 0.1UF 100V X7R 0603" H 4325 3625 50  0001 C CIN "Description"
+F 4 "CAP CER 0.1UF 16V X7R 0603" H 4325 3625 50  0001 C CIN "Description"
 F 5 "Murata" H 4325 3625 50  0001 C CIN "MF_Name"
-F 6 "GRM188R72A104KA35D" H 4325 3625 50  0001 C CIN "MF_PN"
+F 6 "GCM188R71C104KA37D" H 4325 3625 50  0001 C CIN "MF_PN"
 F 7 "Digikey" H 4325 3625 50  0001 C CIN "S1_Name"
-F 8 "490-3285-1-ND" H 4325 3625 50  0001 C CIN "S1_PN"
+F 8 "490-4774-1-ND" H 4325 3625 50  0001 C CIN "S1_PN"
+F 9 "smt" H 0   0   50  0001 C CNN "Type"
+F 10 "114" H 0   0   50  0001 C CNN "XSize_mils"
+F 11 "59" H 0   0   50  0001 C CNN "YSize_mils"
 	1    4325 3975
 	1    0    0    -1
 $EndComp
+Wire Wire Line
+	5550 4625 5550 4700
+Wire Wire Line
+	4325 3775 5050 3775
 $EndSCHEMATC
