File: Circuit-Kits/Modules/2x3-LED-RGB-SMT-Round-Flat-Top/2x3-LED-RGB-SMT-Round-Flat-Top.sch (KiCad schematic (older format))
At the start: 1 part

Commit message: Port project to KiCad 5.0
Parts:
- LED1: symbol LED-RGB-SMT-QBLP600-RGB -> crazy_circuits:LED-RGB-SMT-QBLP600-RGB
Changed lines of the file:
@@
-EESchema Schematic File Version 2
+EESchema Schematic File Version 4
 LIBS:crazy_circuits
-EELAYER 25 0
+EELAYER 26 0
 EELAYER END
 $Descr USLetter 11000 8500
@@
 	4600 3300 4600 3250
 $Comp
-L VCC #PWR01
+L crazy_circuits:VCC #PWR01
 U 1 1 58830E25
 P 4600 3250
@@
 B
 $Comp
-L LED-RGB-SMT-QBLP600-RGB LED1
+L crazy_circuits:LED-RGB-SMT-QBLP600-RGB LED1
 U 1 1 58831339
 P 4750 3525
