File: Circuit-Kits/Modules/2x3-Mini-Potentiometer-3386P-TH/2x3-Mini-Potentiometer-3386P-TH.sch (KiCad schematic (older format))
At the start: 1 part

Commit message: Port project to KiCad 5.0
Parts:
- R1: symbol TRIMPOT-10K-3PIN-TH-3368P-1-103TLF -> crazy_circuits:TRIMPOT-10K-3PIN-TH-3368P-1-103TLF
Changed lines of the file:
@@
-EESchema Schematic File Version 2
+EESchema Schematic File Version 4
 LIBS:crazy_circuits
-LIBS:2x3-Mini-Potentiometer-3386P-TH-cache
-EELAYER 25 0
+EELAYER 26 0
 EELAYER END
 $Descr USLetter 11000 8500
@@
 $EndDescr
 $Comp
-L TRIMPOT-10K-3PIN-TH-3368P-1-103TLF R1
+L crazy_circuits:TRIMPOT-10K-3PIN-TH-3368P-1-103TLF R1
 U 1 1 5882C850
 P 4600 3900
@@
 $EndComp
 $Comp
-L VCC #PWR01
+L crazy_circuits:VCC #PWR01
 U 1 1 5882C895
 P 4600 3650
@@
 	4600 4050 4600 4125
 $Comp
-L GND #PWR02
+L crazy_circuits:GND #PWR02
 U 1 1 5882C8C2
 P 4600 4125
