File: Circuit-Kits/Modules/2x4-Grove-Sensor-Inline/2x4-Grove-Sensor-Inline.sch (KiCad schematic (older format))
At the start: 1 part, among them J1 SEEED GROVE SENSOR

Commit message: Port project to KiCad 5.0
Parts:
- J1: symbol HEADER-MALE-4POS-TH-1x04-SEEED-GROVE -> crazy_circuits:HEADER-MALE-4POS-TH-1x04-SEEED-GROVE
Changed lines of the file:
@@
-EESchema Schematic File Version 2
+EESchema Schematic File Version 4
 LIBS:crazy_circuits
-EELAYER 25 0
+EELAYER 26 0
 EELAYER END
 $Descr USLetter 11000 8500
@@
 $EndDescr
 $Comp
-L HEADER-MALE-4POS-TH-1x04-SEEED-GROVE J1
+L crazy_circuits:HEADER-MALE-4POS-TH-1x04-SEEED-GROVE J1
 U 1 1 5A7DB41E
 P 5225 3275
@@
 	4850 3475 4850 3575
 $Comp
-L GND #PWR01
+L crazy_circuits:GND #PWR01
 U 1 1 5A7DB4D9
 P 4850 3575
@@
 $EndComp
 $Comp
-L VCC #PWR02
+L crazy_circuits:VCC #PWR02
 U 1 1 5A7DB4EF
 P 4850 3025
