File: Circuit-Kits/Modules/5x10-Teensy-LC-Breakout/5x10-Teensy-LC-Breakout.sch (KiCad schematic (older format))
At the start: 1 part, among them U1 Teensy

Commit message: Port project to KiCad 5.0
Parts:
- U1: symbol Teensy -> crazy_circuits:Teensy
Changed lines of the file:
@@
-EESchema Schematic File Version 2
+EESchema Schematic File Version 4
 LIBS:crazy_circuits
-EELAYER 25 0
+EELAYER 26 0
 EELAYER END
 $Descr USLetter 11000 8500
@@
 $EndDescr
 $Comp
-L Teensy U1
+L crazy_circuits:Teensy U1
 U 1 1 5882FEC7
 P 3400 3075
 F 0 "U1" H 3500 3125 50  0000 L CNN
 F 1 "Teensy" H 3500 3025 50  0000 L CNN
-F 2 "Crazy_Circuits:TEENSYLC-5x10-RING" V 3400 3115 50  0000 C CNN
+F 2 "Crazy_Circuits:TEENSYLC-5x10-RING" V 3400 3115 50  0001 C CNN
 F 3 "" V 3400 3115 50  0000 C CNN
 F 4 "TEENSY LC DEVELOPMENT BOARD" H 3400 3075 60  0001 C CNN "Description"
