File: Circuit-Kits/Modules/6x10-Photon-Breakout/6x10-Photon-Breakout.sch (KiCad schematic (older format))
At the start: 1 part, among them U1 PARTICLE-PHOTON-V016

Commit message: Port project to KiCad 5.0
Parts:
- U1: symbol PARTICLE-PHOTON-V016 -> crazy_circuits:PARTICLE-PHOTON-V016
Connections:
- wire segments 24 -> 25
Changed lines of the file:
@@
-EESchema Schematic File Version 2
-LIBS:crazy_circuits
-EELAYER 25 0
+EESchema Schematic File Version 4
+EELAYER 26 0
 EELAYER END
 $Descr USLetter 11000 8500
@@
 $EndDescr
 $Comp
-L PARTICLE-PHOTON-V016 U1
+L crazy_circuits:PARTICLE-PHOTON-V016 U1
 U 1 1 5B4C1D29
 P 2850 3375
@@
 	3050 2025 3400 2025
 Wire Wire Line
-	3400 1900 3400 2225
+	3400 1900 3400 2025
 $Comp
-L 5V #PWR01
+L crazy_circuits:5V #PWR01
 U 1 1 5B4C2204
 P 3400 1900
@@
 	3600 2125 3600 1975
 $Comp
-L 3.3V #PWR02
+L crazy_circuits:3.3V #PWR02
 U 1 1 5B4C222C
 P 3600 1975
@@
 	3700 5175 3700 5300
 $Comp
-L GND #PWR03
+L crazy_circuits:GND #PWR03
 U 1 1 5B4C30DD
 P 3700 5300
@@
 	3400 2225 3050 2225
 Connection ~ 3400 2025
+Wire Wire Line
+	3400 2025 3400 2225
 $EndSCHEMATC
