File: Circuit-Kits/Modules/8x12-PocketBeagle-Breakout/8x12-PocketBeagle-Breakout.sch (KiCad schematic (older format))
At the start: 6 parts, among them J1 HEADER, J2 HEADER, J3 HEADER, J4 HEADER, J5 HEADER, J6 POCKETBEAGLE

Commit message: Port project to KiCad 5.0
Parts:
- J1, J2, J3, J4, J5: symbol HEADER-MALE-3POS-TH-1x03-P0.1IN -> crazy_circuits:HEADER-MALE-3POS-TH-1x03-P0.1IN
- J6: symbol POCKET-BEAGLE -> crazy_circuits:POCKET-BEAGLE
Connections:
- wire segments 53 -> 61
Changed lines of the file:
@@
-EESchema Schematic File Version 2
+EESchema Schematic File Version 4
 LIBS:crazy_circuits
 LIBS:8x12-PocketBeagle-Breakout-cache
-EELAYER 25 0
+EELAYER 26 0
 EELAYER END
 $Descr USLetter 11000 8500
@@
 $EndDescr
 $Comp
-L POCKET-BEAGLE J6
+L crazy_circuits:POCKET-BEAGLE J6
 U 1 1 5B67D22A
 P 4275 4075
@@
 $EndComp
 $Comp
-L HEADER-MALE-3POS-TH-1x03-P0.1IN J4
+L crazy_circuits:HEADER-MALE-3POS-TH-1x03-P0.1IN J4
 U 1 1 5B67D38F
 P 6400 2925
@@
 $EndComp
 $Comp
-L GND #PWR01
+L crazy_circuits:GND #PWR01
 U 1 1 5B67D42B
 P 3425 6025
@@
 $EndComp
 $Comp
-L 5V #PWR02
+L crazy_circuits:5V #PWR02
 U 1 1 5B67DCF4
 P 5000 2025
@@
 $EndComp
 $Comp
-L 3.3V #PWR03
+L crazy_circuits:3.3V #PWR03
 U 1 1 5B67DD0C
 P 5375 2025
@@
 $EndComp
 $Comp
-L GND #PWR04
+L crazy_circuits:GND #PWR04
 U 1 1 5B67DD98
 P 5225 3575
@@
 $EndComp
 $Comp
-L HEADER-MALE-3POS-TH-1x03-P0.1IN J5
+L crazy_circuits:HEADER-MALE-3POS-TH-1x03-P0.1IN J5
 U 1 1 5B67DF01
 P 6400 3425
@@
 $EndComp
 Wire Wire Line
-	3425 5575 3425 6025
+	3425 5575 3425 5675
 Wire Wire Line
 	3425 5575 3625 5575
@@
 	5375 2625 4875 2625
 Wire Wire Line
-	5375 2025 5375 2625
+	5375 2025 5375 2325
 Wire Wire Line
 	4875 2325 5375 2325
@@
 	4875 2125 5000 2125
 Wire Wire Line
-	5000 2025 5000 2225
+	5000 2025 5000 2125
 Wire Wire Line
 	5000 2225 4875 2225
@@
 	6200 2925 5950 2925
 Wire Wire Line
-	5950 2725 5950 3425
-$Comp
-L 3.3V #PWR05
+	5950 2725 5950 2925
+$Comp
+L crazy_circuits:3.3V #PWR05
 U 1 1 5B67E125
 P 5950 2725
@@
 	6200 3025 6050 3025
 Wire Wire Line
-	6050 3025 6050 3700
+	6050 3025 6050 3525
 Wire Wire Line
 	6200 3525 6050 3525
 Connection ~ 6050 3525
 $Comp
-L GND #PWR06
+L crazy_circuits:GND #PWR06
 U 1 1 5B67E1BE
 P 6050 3700
@@
 NoConn ~ 3625 2375
 $Comp
-L HEADER-MALE-3POS-TH-1x03-P0.1IN J1
+L crazy_circuits:HEADER-MALE-3POS-TH-1x03-P0.1IN J1
 U 1 1 5B687160
 P 6400 5325
@@
 $EndComp
 $Comp
-L HEADER-MALE-3POS-TH-1x03-P0.1IN J2
+L crazy_circuits:HEADER-MALE-3POS-TH-1x03-P0.1IN J2
 U 1 1 5B68720A
 P 6400 4125
@@
 	5775 4125 5775 3925
 $Comp
-L 5V #PWR07
+L crazy_circuits:5V #PWR07
 U 1 1 5B687399
 P 5775 3925
@@
 $EndComp
 $Comp
-L GND #PWR08
+L crazy_circuits:GND #PWR08
 U 1 1 5B6873B7
 P 6200 4350
@@
 	6075 5325 6075 5150
 $Comp
-L 5V #PWR09
+L crazy_circuits:5V #PWR09
 U 1 1 5B68744D
 P 6075 5150
@@
 	6075 5425 6075 5550
 $Comp
-L GND #PWR010
+L crazy_circuits:GND #PWR010
 U 1 1 5B6874AA
 P 6075 5550
@@
 $EndComp
 $Comp
-L HEADER-MALE-3POS-TH-1x03-P0.1IN J3
+L crazy_circuits:HEADER-MALE-3POS-TH-1x03-P0.1IN J3
 U 1 1 5B68755C
 P 2350 4625
@@
 	2675 4625 2675 4475
 $Comp
-L 5V #PWR011
+L crazy_circuits:5V #PWR011
 U 1 1 5B6876D8
 P 2675 4475
@@
 	2675 4725 2675 4775
 $Comp
-L GND #PWR012
+L crazy_circuits:GND #PWR012
 U 1 1 5B68773C
 P 2675 4775
@@
 	1    0    0    -1
 $EndComp
+Wire Wire Line
+	3425 5675 3425 5775
+Wire Wire Line
+	3425 5775 3425 5875
+Wire Wire Line
+	3425 5875 3425 6025
+Wire Wire Line
+	5375 2325 5375 2425
+Wire Wire Line
+	5375 2425 5375 2625
+Wire Wire Line
+	5000 2125 5000 2225
+Wire Wire Line
+	5950 2925 5950 3425
+Wire Wire Line
+	6050 3525 6050 3700
 $EndSCHEMATC
