File: Circuit-Kits/Modules/1x3-Button-Momentary/1x3-Button-Momentary.sch (KiCad schematic (older format))
At the start: 1 part, among them SW1 SW_PUSH

Commit message: Port project to KiCad 5.0
Parts:
- SW1: symbol SW_PUSH -> crazy_circuits:SW_PUSH
Changed lines of the file:
@@
-EESchema Schematic File Version 2
+EESchema Schematic File Version 4
 LIBS:crazy_circuits
-LIBS:1x3-Button-Momentary-cache
-EELAYER 25 0
+EELAYER 26 0
 EELAYER END
 $Descr USLetter 11000 8500
@@
 $EndDescr
 $Comp
-L SW_PUSH SW1
+L crazy_circuits:SW_PUSH SW1
 U 1 1 585732B9
 P 4375 3450

Commit message: Adjust silk, copper. Release 1x3 Momentary TH v1.3
Parts:
- SW1: Type (none) -> th; XSize_mils (none) -> 237; YSize_mils (none) -> 237
Changed lines of the file:
@@
 EESchema Schematic File Version 4
 LIBS:crazy_circuits
+LIBS:1x3-Button-Momentary-cache
 EELAYER 26 0
 EELAYER END
@@
 Title "1x3 Momentary Pushbutton Module"
 Date "18 Dec 2016"
-Rev "1.0"
+Rev "v1.3"
 Comp "CERN Open Hardware License v1.2."
 Comment1 "help@browndoggadgets.com"
@@
 F 7 "Digikey" H 4375 3450 60  0001 C CNN "S1_Name"
 F 8 "SW400-ND" H 4375 3450 60  0001 C CNN "S1_PN"
+F 9 "237" H 4375 3450 50  0001 C CNN "XSize_mils"
+F 10 "237" H 4375 3450 50  0001 C CNN "YSize_mils"
+F 11 "th" H 4375 3450 50  0001 C CNN "Type"
 	1    4375 3450
 	1    0    0    -1

Commit message: Update symbol data, no revision.
Parts:
- removed SW1: SW_PUSH, Crazy_Circuits:BUTTON-1x3-TH-OMRON-B3F-1XXX, symbol crazy_circuits:SW_PUSH
- added SW1: SWITCH-PUSH-MOMENT-TH-B3F-1000, Crazy_Circuits:BUTTON-1x3-TH-OMRON-B3F-1XXX, symbol crazy_circuits:SWITCH-MOMENT-SPDT-TH-B3F-1000
Connections:
- wire segments 2 -> 8
Changed lines of the file:
@@
 Comment4 ""
 $EndDescr
+Wire Wire Line
+	4075 3450 4050 3450
+Wire Wire Line
+	4675 3450 4700 3450
+Text Label 4825 3450 2    50   ~ 0
+2
+Text Label 3925 3450 0    50   ~ 0
+1
 $Comp
-L crazy_circuits:SW_PUSH SW1
-U 1 1 585732B9
+L crazy_circuits:SWITCH-MOMENT-SPDT-TH-B3F-1000 SW1
+U 1 1 5BAAC142
 P 4375 3450
-F 0 "SW1" H 4525 3560 50  0000 C CNN
-F 1 "SW_PUSH" H 4375 3370 50  0000 C CNN
-F 2 "Crazy_Circuits:BUTTON-1x3-TH-OMRON-B3F-1XXX" H 4375 3450 50  0001 C CNN
-F 3 "" H 4375 3450 50  0000 C CNN
-F 4 "SWITCH TACTILE SPST-NO 0.05A 24V" H 4375 3450 60  0001 C CNN "Description"
-F 5 "Omron" H 4375 3450 60  0001 C CNN "MF_Name"
-F 6 "B3F-1000" H 4375 3450 60  0001 C CNN "MF_PN"
-F 7 "Digikey" H 4375 3450 60  0001 C CNN "S1_Name"
-F 8 "SW400-ND" H 4375 3450 60  0001 C CNN "S1_PN"
-F 9 "237" H 4375 3450 50  0001 C CNN "XSize_mils"
-F 10 "237" H 4375 3450 50  0001 C CNN "YSize_mils"
-F 11 "th" H 4375 3450 50  0001 C CNN "Type"
+F 0 "SW1" H 4375 3705 50  0000 C CNN
+F 1 "SWITCH-PUSH-MOMENT-TH-B3F-1000" H 4375 3614 50  0000 C CNN
+F 2 "Crazy_Circuits:BUTTON-1x3-TH-OMRON-B3F-1XXX" H 4375 3250 50  0001 C CIN
+F 3 "http://www.omron.com/ecb/products/pdf/en-b3fs_4.pdf" H 4375 3450 10  0001 C CNN
+F 4 "SWITCH MOMENT SPST-NO 0.05A 24V SMT B3F-1000" H 4375 3250 50  0001 C CIN "Description"
+F 5 "Omron" H 4375 3250 50  0001 C CIN "MF_Name"
+F 6 "B3F-1000" H 4375 3250 50  0001 C CIN "MF_PN"
+F 7 "Digikey" H 4375 3250 50  0001 C CIN "S1_Name"
+F 8 "SW400-ND" H 4375 3250 50  0001 C CIN "S1_PN"
+F 9 "237" H 4375 3260 50  0001 C CNN "XSize_mils"
+F 10 "237" H 4375 3260 50  0001 C CNN "YSize_mils"
+F 11 "th" H 4375 3260 50  0001 C CNN "Type"
 	1    4375 3450
 	1    0    0    -1
 $EndComp
 Wire Wire Line
-	4075 3450 3925 3450
+	4050 3450 4050 3550
 Wire Wire Line
-	4675 3450 4825 3450
-Text Label 4825 3450 2    50   ~ 0
-2
-Text Label 3925 3450 0    50   ~ 0
-1
+	4050 3550 4075 3550
+Connection ~ 4050 3450
+Wire Wire Line
+	4050 3450 3925 3450
+Wire Wire Line
+	4675 3550 4700 3550
+Wire Wire Line
+	4700 3550 4700 3450
+Connection ~ 4700 3450
+Wire Wire Line
+	4700 3450 4825 3450
 $EndSCHEMATC
