File: Circuit-Kits/Modules/1x3-Button-Momentary-SMT/1x3-Button-Momentary-SMT.kicad_pcb (KiCad board)
At the start: 2 copper layers, 23.5 x 7.6 mm, 1 part, among them SW1 PTS645

Commit message: Update silk, copper. Release 1x3 Button SMT v1.2
Changed lines of the file:
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@@
-(kicad_pcb (version 4) (host pcbnew 4.0.5-e0-6337~49~ubuntu16.04.1)
+(kicad_pcb (version 20171130) (host pcbnew 5.0.0-fee4fd1~66~ubuntu16.04.1)
   (general
-    (links 4)
-    (no_connects 4)
-    (area 0.127 23.07 142.971759 121.412)
     (thickness 1.6)
     (drawings 1)
@@
     (title "1x3 Momentary Pushbutton SMT Module")
     (date "23 May 2017")
-    (rev v1.1)
+    (rev "v1.2")
     (company "CERN Open Hardware License v1.2.")
-    (comment 1 help@browndoggadgets.com)
-    (comment 2 http://browndoggadgets.com/)
+    (comment 1 "help@browndoggadgets.com")
+    (comment 2 "http://browndoggadgets.com/")
     (comment 3 "Brown Dog Gadgets")
   )
@@
       (layerselection 0x310fc_80000001)
       (usegerberextensions true)
+      (usegerberattributes false)
+      (usegerberadvancedattributes false)
+      (creategerberjobfile false)
       (excludeedgelayer true)
       (linewidth 0.100000)
@@
       (hpglpennumber 1)
       (hpglpenspeed 20)
-      (hpglpendiameter 15)
-      (hpglpenoverlay 2)
+      (hpglpendiameter 15.000000)
       (psnegative false)
       (psa4output false)
@@
       (drillshape 0)
       (scaleselection 1)
-      (outputdirectory gerbers))
+      (outputdirectory "gerbers"))
   )
   (net 0 "")
@@
       (effects (font (size 1 1) (thickness 0.15)))
     )
+    (fp_arc (start 0 0) (end 1.3 -2.4) (angle -230.6919655) (layer F.Mask) (width 0.8))
+    (fp_arc (start 16 0) (end 14.7 2.4) (angle -230.6919655) (layer F.Mask) (width 0.8))
     (fp_line (start 2.286 -2.286) (end 0 0) (layer F.Cu) (width 0.5))
     (fp_line (start 4.064 -2.286) (end 2.286 -2.286) (layer F.Cu) (width 0.5))
-    (fp_line (start 12.0142 -3.5052) (end 12.0142 3.7846) (layer F.SilkS) (width 0.1))
-    (fp_line (start 3.9878 3.81) (end 3.9878 -3.5052) (layer F.SilkS) (width 0.1))
     (fp_line (start 11.0254 3.0456) (end 5.0254 3.0456) (layer F.Fab) (width 0.04064))
     (fp_line (start 11.0254 -2.9544) (end 11.0254 3.0456) (layer F.Fab) (width 0.04064))
     (fp_line (start 5.0254 -2.9544) (end 11.0254 -2.9544) (layer F.Fab) (width 0.04064))
     (fp_line (start 5.0254 3.0456) (end 5.0254 -2.9544) (layer F.Fab) (width 0.04064))
-    (fp_arc (start 0.106632 -0.00018) (end -3.693368 0.09982) (angle 89.9) (layer Edge.Cuts) (width 0.04064))
-    (fp_arc (start 0.111824 0) (end 0 3.8) (angle 88.31442243) (layer Edge.Cuts) (width 0.04064))
-    (fp_arc (start 16 0) (end 19.8 -0.1) (angle 91.50743576) (layer Edge.Cuts) (width 0.04064))
-    (fp_arc (start 16 0) (end 15.9 -3.8) (angle 91.50743576) (layer Edge.Cuts) (width 0.04064))
-    (fp_line (start 15.9 -3.8) (end 0 -3.8) (layer Edge.Cuts) (width 0.04064))
-    (fp_line (start 16.1 3.8) (end 0 3.8) (layer Edge.Cuts) (width 0.04064))
+    (fp_arc (start 0.106632 -0.00018) (end -3.693368 0.09982) (angle 89.9) (layer Edge.Cuts) (width 0.08))
+    (fp_arc (start 0.111824 0) (end 0 3.8) (angle 88.31442243) (layer Edge.Cuts) (width 0.08))
+    (fp_arc (start 16 0) (end 19.8 -0.1) (angle 91.50743576) (layer Edge.Cuts) (width 0.08))
+    (fp_arc (start 16 0) (end 15.9 -3.8) (angle 91.50743576) (layer Edge.Cuts) (width 0.08))
+    (fp_line (start 15.9 -3.8) (end 0 -3.8) (layer Edge.Cuts) (width 0.08))
+    (fp_line (start 16.1 3.8) (end 0 3.8) (layer Edge.Cuts) (width 0.08))
     (fp_arc (start 0.106632 -0.00018) (end -3.693368 0.09982) (angle 89.9) (layer F.Fab) (width 0.04064))
     (fp_arc (start 0.111824 0) (end 0 3.8) (angle 88.31442243) (layer F.Fab) (width 0.04064))
@@
     (fp_line (start 15.9 -3.8) (end 0 -3.8) (layer F.Fab) (width 0.04064))
     (fp_line (start 16 3.8) (end 0 3.8) (layer F.Fab) (width 0.04064))
-    (fp_line (start 16.102 0.0238) (end 16.002 -0.0762) (layer F.SilkS) (width 7.2))
+    (fp_line (start 16.102 0.0238) (end 16.002 -0.0762) (layer F.SilkS) (width 7.5))
     (fp_line (start 11.938 2.286) (end 13.716 2.286) (layer F.Cu) (width 0.5))
     (fp_line (start 13.716 2.286) (end 16.002 0) (layer F.Cu) (width 0.5))
-    (pad 1 thru_hole circle (at 0 0 270) (size 6 6) (drill 4.98) (layers *.Cu *.Mask)
+    (pad 1 thru_hole circle (at 0 0 270) (size 6.2 6.2) (drill 4.98) (layers *.Cu B.Mask)
       (net 1 /1) (solder_mask_margin 0.0254))
     (pad "" np_thru_hole circle (at 8 0 270) (size 4.98 4.98) (drill 4.98) (layers *.Cu))
@@
     (pad 2 smd rect (at 11.9754 -2.1544) (size 1.55 1.3) (layers F.Cu F.Paste F.Mask)
       (net 1 /1) (solder_mask_margin 0.0762))
-    (pad 2 thru_hole circle (at 16 0 270) (size 6 6) (drill 4.98) (layers *.Cu *.Mask)
+    (pad 2 thru_hole circle (at 16 0 270) (size 6.2 6.2) (drill 4.98) (layers *.Cu B.Mask)
       (net 1 /1) (solder_mask_margin 0.0254))
   )
