File: Circuit-Kits/Modules/1x3-Button-Momentary-SMT/1x3-Button-Momentary-SMT.sch (KiCad schematic (older format))
At the start: 1 part, among them SW1 PTS645

Commit message: Port project to KiCad 5.0
Parts:
- SW1: symbol SWITCH-MOMENT-SPDT-SMT-B3FS-4002P -> crazy_circuits:SWITCH-MOMENT-SPDT-SMT-B3FS-4002P
Connections:
- wire segments 6 -> 8
Changed lines of the file:
@@
-EESchema Schematic File Version 2
+EESchema Schematic File Version 4
 LIBS:crazy_circuits
-EELAYER 25 0
+EELAYER 26 0
 EELAYER END
 $Descr USLetter 11000 8500
@@
 $EndDescr
 $Comp
-L SWITCH-MOMENT-SPDT-SMT-B3FS-4002P SW1
+L crazy_circuits:SWITCH-MOMENT-SPDT-SMT-B3FS-4002P SW1
 U 1 1 5877E7CA
 P 4875 3625
@@
 	4525 3725 4525 3625
 Wire Wire Line
-	4400 3625 4575 3625
+	4400 3625 4525 3625
 Connection ~ 4525 3625
 Text Label 4400 3625 0    50   ~ 0
 1
 Wire Wire Line
-	5175 3625 5325 3625
+	5175 3625 5225 3625
 Wire Wire Line
 	5175 3725 5225 3725
@@
 Text Label 5325 3625 2    50   ~ 0
 2
+Wire Wire Line
+	4525 3625 4575 3625
+Wire Wire Line
+	5225 3625 5325 3625
 $EndSCHEMATC

Commit message: Update silk, copper. Release 1x3 Button SMT v1.2
Parts:
- removed SW1: PTS645, Crazy_Circuits:SWITCH-6mm-SQUARE-PTS645-SMT-1x3, symbol crazy_circuits:SWITCH-MOMENT-SPDT-SMT-B3FS-4002P
- added SW1: P/N PTS645, Wickerlib:SWITCH-OMRON-MOMENTARY-SMT-B3FS-4000, symbol crazy_circuits:SWITCH-MOMENT-SPDT-SMT-PTS645
Changed lines of the file:
@@
 EESchema Schematic File Version 4
 LIBS:crazy_circuits
+LIBS:1x3-Button-Momentary-SMT-cache
 EELAYER 26 0
 EELAYER END
@@
 Comment4 ""
 $EndDescr
-$Comp
-L crazy_circuits:SWITCH-MOMENT-SPDT-SMT-B3FS-4002P SW1
-U 1 1 5877E7CA
-P 4875 3625
-F 0 "SW1" H 5025 3735 50  0000 C CNN
-F 1 "PTS645" H 4845 3425 50  0000 C CNN
-F 2 "Crazy_Circuits:SWITCH-6mm-SQUARE-PTS645-SMT-1x3" H 4875 3275 50  0001 C CIN
-F 3 "http://www.omron.com/ecb/products/pdf/en-b3fs_4.pdf" H 4875 3625 10  0001 C CNN
-F 4 "SWITCH MOMENT SPST-NO 0.05A 14V SMT PTS645" H 4875 3275 50  0001 C CIN "Description"
-F 5 "C&K" H 4875 3275 50  0001 C CIN "MF_Name"
-F 6 "PTS645SM43SMTR92 LFS" H 4875 3275 50  0001 C CIN "MF_PN"
-F 7 "Digikey" H 4875 3275 50  0001 C CIN "S1_Name"
-F 8 "CKN9112TR-ND" H 4875 3275 50  0001 C CIN "S1_PN"
-	1    4875 3625
-	1    0    0    -1
-$EndComp
 Wire Wire Line
 	4575 3725 4525 3725
@@
 Wire Wire Line
 	5225 3625 5325 3625
+$Comp
+L crazy_circuits:SWITCH-MOMENT-SPDT-SMT-PTS645 SW1
+U 1 1 5BA9E78D
+P 4875 3625
+F 0 "SW1" H 4875 3775 50  0000 C CNN
+F 1 "P/N PTS645" H 4875 3425 50  0000 C CNN
+F 2 "Wickerlib:SWITCH-OMRON-MOMENTARY-SMT-B3FS-4000" H 4875 3275 50  0001 C CIN
+F 3 "https://www.ckswitches.com/media/1471/pts645.pdf" H 4875 3625 10  0001 C CNN
+F 4 "SWITCH MOMENT SPST-NO 0.05A 12V SMT PTS645" H 4875 3275 50  0001 C CIN "Description"
+F 5 "C&K" H 4875 3275 50  0001 C CIN "MF_Name"
+F 6 "PTS645SM43SMTR92 LFS" H 4875 3275 50  0001 C CIN "MF_PN"
+F 7 "Digikey" H 4875 3275 50  0001 C CIN "S1_Name"
+F 8 "CKN9112CT-ND" H 4875 3275 50  0001 C CIN "S1_PN"
+F 9 "237" H 4725 3285 50  0001 C CNN "XSize_mils"
+F 10 "237" H 4875 3285 50  0001 C CNN "YSize_mils"
+F 11 "smt" H 4975 3285 50  0001 C CNN "Type"
+	1    4875 3625
+	1    0    0    -1
+$EndComp
 $EndSCHEMATC
