File: Circuit-Kits/Modules/2x3-Servo-Header/2x3-Servo-Header.sch (KiCad schematic (older format))
At the start: 1 part, among them J1 Servo_Breakout

Commit message: Update symbol data, no revision.
Parts:
- J1: symbol crazy_circuits:Servo_Breakout -> crazy_circuits:HEADER-MALE-SERVO-3PIN-1x3-TH; Type (none) -> th; XSize_mils (none) -> 100; YSize_mils (none) -> 300
Changed lines of the file:
@@
 EESchema Schematic File Version 4
 LIBS:crazy_circuits
+LIBS:2x3-Servo-Header-cache
 EELAYER 26 0
 EELAYER END
@@
 $EndDescr
 $Comp
-L crazy_circuits:Servo_Breakout J1
+L crazy_circuits:HEADER-MALE-SERVO-3PIN-1x3-TH J1
 U 1 1 588073C1
 P 5175 4300
@@
 F 7 "Digikey" H 5175 4300 60  0001 C CNN "S1_Name"
 F 8 "732-5316-ND" H 5175 4300 60  0001 C CNN "S1_PN"
+F 9 "100" H 0   0   50  0001 C CNN "XSize_mils"
+F 10 "300" H 0   0   50  0001 C CNN "YSize_mils"
+F 11 "th" H 0   0   50  0001 C CNN "Type"
 	1    5175 4300
 	1    0    0    -1

Commit message: Release 2x3 Female Servo Module v1.0
Parts:
- J1: symbol crazy_circuits:HEADER-MALE-SERVO-3PIN-1x3-TH -> 2x3-Servo-Header-rescue:HEADER-MALE-SERVO-3PIN-1x3-TH-crazy_circuits
Changed lines of the file:
@@
 $EndDescr
 $Comp
-L crazy_circuits:HEADER-MALE-SERVO-3PIN-1x3-TH J1
+L 2x3-Servo-Header-rescue:HEADER-MALE-SERVO-3PIN-1x3-TH-crazy_circuits J1
 U 1 1 588073C1
 P 5175 4300
