File: Circuit-Kits/Modules/3x3-CR2032-Coin-Cell/3x3-CR2032-Coin-Cell.sch (KiCad schematic (older format))
At the start: 1 part

Commit message: Port project to KiCad 5.0
Parts:
- BT1: symbol Battery -> crazy_circuits:Battery
Changed lines of the file:
@@
-EESchema Schematic File Version 2
+EESchema Schematic File Version 4
 LIBS:crazy_circuits
-LIBS:3x3-CR2032-Coin-Cell-cache
-EELAYER 25 0
+EELAYER 26 0
 EELAYER END
 $Descr USLetter 11000 8500
@@
 $EndDescr
 $Comp
-L Battery BT1
+L crazy_circuits:Battery BT1
 U 1 1 5858515E
 P 4825 3700
@@
 $EndComp
 $Comp
-L GND #PWR01
+L crazy_circuits:GND #PWR01
 U 1 1 5858519B
 P 4825 3975
@@
 	4825 3550 4825 3375
 $Comp
-L VCC #PWR02
+L crazy_circuits:VCC #PWR02
 U 1 1 585851B9
 P 4825 3375

Commit message: Change silk, copper. Release CR2032 3x3 v1.3
Parts:
- BT1: Type (none) -> smt
Changed lines of the file:
@@
 EESchema Schematic File Version 4
 LIBS:crazy_circuits
+LIBS:3x3-CR2032-Coin-Cell-cache
 EELAYER 26 0
 EELAYER END
@@
 Title "3x3 CR2032 Coin Cell Battery Module"
 Date "19 Dec 2016"
-Rev "1.0"
+Rev "v1.3"
 Comp "CERN Open Hardware License v1.2."
 Comment1 "help@browndoggadgets.com"
@@
 F 7 "Digikey" H 4825 3700 60  0001 C CNN "S1_Name"
 F 8 "BK-912-ND" H 4825 3700 60  0001 C CNN "S1_PN"
+F 9 "smt" H 4825 3700 50  0001 C CNN "Type"
 	1    4825 3700
 	1    0    0    -1
