File: Circuit-Kits/Modules/3x4-CR2032-Coin-Cell-Magnet/3x4-CR2032-Coin-Cell-Magnet.sch (KiCad schematic (older format))
At the start: 1 part

Commit message: Port project to KiCad 5.0
Parts:
- BT1: symbol Battery -> crazy_circuits:Battery
Changed lines of the file:
@@
-EESchema Schematic File Version 2
+EESchema Schematic File Version 4
 LIBS:crazy_circuits
-LIBS:3x4-CR2032-Coin-Cell-Magnet-cache
-EELAYER 25 0
+EELAYER 26 0
 EELAYER END
 $Descr USLetter 11000 8500
@@
 $EndDescr
 $Comp
-L Battery BT1
+L crazy_circuits:Battery BT1
 U 1 1 5858515E
 P 4850 3450
@@
 $EndComp
 $Comp
-L VCC #PWR01
+L crazy_circuits:VCC #PWR01
 U 1 1 58585371
 P 4850 3200
@@
 	4850 3600 4850 3700
 $Comp
-L GND #PWR02
+L crazy_circuits:GND #PWR02
 U 1 1 5858538F
 P 4850 3700

Commit message: Change silk, copper. Release CR2032 3x4 Magnet v1.3
Parts:
- BT1: Type (none) -> smt
Changed lines of the file:
@@
 EESchema Schematic File Version 4
 LIBS:crazy_circuits
+LIBS:3x4-CR2032-Coin-Cell-Magnet-cache
 EELAYER 26 0
 EELAYER END
@@
 encoding utf-8
 Sheet 1 1
-Title "4x3 CR2032 Coin Cell Battery Module"
+Title "3x4 CR2032 Coin Cell Battery Module"
 Date "19 Dec 2016"
-Rev "1.0"
+Rev "v1.3"
 Comp "CERN Open Hardware License v1.2."
 Comment1 "help@browndoggadgets.com"
@@
 F 7 "Digikey" H 4850 3450 60  0001 C CNN "S1_Name"
 F 8 "BK-912-ND" H 4850 3450 60  0001 C CNN "S1_PN"
+F 9 "smt" H 4850 3450 50  0001 C CNN "Type"
 	1    4850 3450
 	1    0    0    -1
