File: Circuit-Kits/Modules/3x4-CR2032-Coin-Cell-On-Off-Switch/3x4-CR2032-Coin-Cell-On-Off-Switch.sch (KiCad schematic (older format))
At the start: 2 parts

Commit message: Port project to KiCad 5.0
Parts:
- BT1: symbol BATT-CR2023-SMT-BK-912 -> crazy_circuits:BATT-CR2023-SMT-BK-912
- S1: symbol SWITCH-SLIDE-SPDT-200MA-30V-EG1218 -> crazy_circuits:SWITCH-SLIDE-SPDT-200MA-30V-EG1218
Changed lines of the file:
@@
-EESchema Schematic File Version 2
+EESchema Schematic File Version 4
 LIBS:crazy_circuits
 LIBS:wickerlib
-LIBS:3x4-CR2032-Coin-Cell-On-Off-Switch-cache
-EELAYER 25 0
+EELAYER 26 0
 EELAYER END
 $Descr USLetter 11000 8500
@@
 $EndDescr
 $Comp
-L VCC #PWR01
+L crazy_circuits:VCC #PWR01
 U 1 1 5B69DD4D
 P 3950 3075
@@
 $EndComp
 $Comp
-L GND #PWR02
+L crazy_circuits:GND #PWR02
 U 1 1 5B69DE1F
 P 4875 3925
@@
 NoConn ~ 4200 3300
 $Comp
-L SWITCH-SLIDE-SPDT-200MA-30V-EG1218 S1
+L crazy_circuits:SWITCH-SLIDE-SPDT-200MA-30V-EG1218 S1
 U 1 1 5B69E7DF
 P 4350 3250
@@
 $EndComp
 $Comp
-L BATT-CR2023-SMT-BK-912 BT1
+L crazy_circuits:BATT-CR2023-SMT-BK-912 BT1
 U 1 1 5B69F74C
 P 4875 3625

Commit message: Change silk, copper. Release CR2032 3x4 Switch v1.1
Parts:
- BT1: Type (none) -> smt
- S1: Type (none) -> th
Changed lines of the file:
@@
 LIBS:crazy_circuits
 LIBS:wickerlib
+LIBS:3x4-CR2032-Coin-Cell-On-Off-Switch-cache
 EELAYER 26 0
 EELAYER END
@@
 Title "3x4 CR2032 Coin Cell On/Off Switch"
 Date "07 Aug 2018"
-Rev "1.0"
+Rev "v1.1"
 Comp "All rights reserved."
 Comment1 "help@browndoggadgets.com"
@@
 F 7 "Digikey" H 4350 2900 50  0001 C CIN "S1_Name"
 F 8 "EG1903-ND" H 4350 2900 50  0001 C CIN "S1_PN"
+F 9 "th" H 4350 3250 50  0001 C CNN "Type"
 	1    4350 3250
 	1    0    0    -1
@@
 F 7 "Digikey" H 4875 3275 50  0001 C CIN "S1_Name"
 F 8 "BK-912-ND" H 4875 3275 50  0001 C CIN "S1_PN"
+F 9 "smt" H 4875 3625 50  0001 C CNN "Type"
 	1    4875 3625
 	1    0    0    -1
